File: BitReactor/schematics/Bit Reactor modular.sch (EAGLE design)
At the start: 111 parts, among them U1 ADC0808N, U2 4053D, U3 4053D, U4 741G3157DBVR, U5 TL072D, U6 LM3914N, U7 LM555D, U9 TL072D

Commit message: v1.2 from Ryan
Parts:
- removed JP1: (no value), jumper:JP1E
- removed R66: 50k, Rebel:POT-ALPS-RK09L1140
- removed U9: TL072D, linear:TL072D
- added C15, C16: 10u, resistor:CPOL-USE2-5
- added C17: 0.01uF, resistor:C-EUC0402
- added IC1: TL074D, linear:TL074D
- C1, C8: device rcl:CPOL-EUE5-6 -> resistor:CPOL-USE2-5
- C4: value 220pF -> 470pF
- R1, R16, R18, R2, R3, R4, R5, R6, R7, R8: value 2.26k -> 20k
- R10, R14, R15: value 1.13k -> 10k; device resistor:R-US_R0805W -> resistor:R-US_R0805
- R11, R12, R13, R9: value 1.13k -> 10k
- R17: value 2.26k -> 2.7K
- R19, R21, R22, R23: value 2.26k -> 10K; device resistor:R-US_R0805 -> Rebel:POT-ALPS-RK09L1140
- R20: value 2.26k -> 50k; device resistor:R-US_R0805 -> Rebel:POT-ALPS-RK09L1140
- R34: device resistor:R-US_R0402 -> resistor:R-US_R0805
- R36: value 10k -> 100k
- R54: value 120k -> 10k; device resistor:R-US_R0402 -> resistor:R-US_R0805
- R62, R63: value POT-ALPS-RK09L1140 -> 120K; device Rebel:POT-ALPS-RK09L1140 -> resistor:R-US_R0402
- R64, R65: value POT-ALPS-RK09L1140 -> 120k; device Rebel:POT-ALPS-RK09L1140 -> resistor:R-US_R0402
Connections:
- removed net N$64: R14.2, R7.1, U2A.X
- removed net N$67: R23.1, U4G$1.B
- removed net N$74: R56.1, R63G$1.2
- new net N$68: C16.+, R34.2
- new net N$85: R15.1, R16.1, U2A.X
- net +12V: now also IC1P.V+, R17.2, R22G$1.1; no longer R62G$1.3, R64G$1.3, U9P.V+
- net -12V: now also IC1P.V-; no longer U9P.V-
- net CV2IN: now also IC1C.OUT; no longer U9A.OUT
- net GND: now also C16.-, C17.1, IC1A.+IN, IC1B.+IN, IC1C.+IN, IC1D.+IN, R19G$1.3, R21G$1.1, R22G$1.3, R23G$1.1; no longer R17.2, R18.2, R19.2, R20.2, R21.2, R22.2, R23.2, R62G$1.1, R63G$1.1, R64G$1.1, R65G$1.1, U9A.+IN, U9B.+IN
- net N$10: now also AUDIOIN.3, C15.+; no longer R10.2, R3.1, U3A.Y
- net N$11: now also C15.-, R36.2; no longer R11.2, R4.1, U3A.X
- net N$12: now also R13.1, R14.2, U2A.Y1; no longer R12.2, R5.1
- net N$13: now also R5.1; no longer R12.1
- net N$14: now also R4.1; no longer R11.1
- net N$15: now also R3.1; no longer R10.1
- net N$16: now also R2.1; no longer R9.1
- net N$17: now also R8.1; no longer R15.1
- net N$18: now also R21G$1.2, R62.1; no longer R15.2, R16.1, R8.1
- net N$19: now also IC1A.-IN, R62.2, R63.1; no longer R17.1, U2A.X1
- net N$20: now also R18.2, R20G$1.1, R34.1; no longer R34.2, R66G$1.1
- net N$21: now also R7.1; no longer R14.1
- net N$22: now also R6.1; no longer R13.1
- net N$23: now also IC1A.OUT, R56.1, R63.2; no longer R18.1, U2A.Y1
- net N$24: now also R12.1, R13.2, U3A.X; no longer R19.1
- net N$25: now also R11.1, R12.2, U3A.Y; no longer R20.1
- net N$26: now also R10.1, R11.2, U3A.Z; no longer R21.1
- net N$27: now also R10.2, R9.1, U4G$1.X; no longer R22.1
- net N$28: now also R9.2, U4G$1.B; no longer U4G$1.X
- net N$38: now also R18.1; no longer R34.1
- net N$40: now also R20G$1.2, R20G$1.3; no longer R66G$1.2, R66G$1.3
- net N$42: now also R23G$1.2, R64.2; no longer AUDIOIN.3, R36.2
- net N$45: now also U1A.START; no longer JP1.2
- net N$47: now also IC1B.-IN, R64.1, R65.2; no longer R53.2, R65G$1.2
- net N$48: now also R23G$1.3; no longer R65G$1.3
- net N$49: now also IC1B.OUT, R53.2, R65.1; no longer JP1.1, U1A.START
- net N$65: now also R14.1, R15.2, U2A.X1; no longer R13.2, R6.1
- net N$71: now also IC1D.-IN; no longer U9B.-IN
- net N$72: now also R19G$1.2; no longer R62G$1.2
- net N$73: now also IC1D.OUT; no longer U9B.OUT
- net N$75: now also R21G$1.3; no longer R63G$1.3
- net N$80: now also C17.2
- net N$81: now also IC1C.-IN; no longer U9A.-IN
- net N$83: now also R22G$1.2; no longer R64G$1.2
- net N$9: now also R17.1, R19G$1.1; no longer R2.1, R9.2, U3A.Z
Other:
- note removed: "+ DC bias here puts CV out of operating range"
- note removed: "DC coupling: 0-10V max out"
- note removed: "must limit to range of -0.3 --> 5.3V"
- moved on the sheet: CRUSH_CV, R10, R11, R12, R13, R14, R15, R16, R17, R18, R34, R55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

Commit message: tied pot shells to gnd
Connections:
- net GND: now also R19G$2.P$1, R20G$2.P$1, R21G$2.P$1, R22G$2.P$1, R23G$2.P$1
Changed lines of the file:
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@@
 <instance part="R32" gate="G$1" x="-66.04" y="-12.7" rot="R90"/>
 <instance part="R33" gate="G$1" x="-55.88" y="-12.7" rot="R90"/>
-<instance part="GND12" gate="1" x="-66.04" y="-22.86"/>
+<instance part="GND12" gate="1" x="-66.04" y="-27.94"/>
 <instance part="R18" gate="G$1" x="-33.02" y="10.16" rot="R180"/>
 <instance part="R36" gate="G$1" x="-78.74" y="0" rot="R180"/>
@@
 <instance part="GND15" gate="1" x="-218.44" y="83.82"/>
 <instance part="GND19" gate="1" x="-121.92" y="76.2"/>
-<instance part="GND21" gate="1" x="-149.86" y="137.16" rot="R180"/>
+<instance part="GND21" gate="1" x="-149.86" y="142.24" rot="R180"/>
 <instance part="GND22" gate="1" x="-208.28" y="83.82"/>
 <instance part="P+5" gate="1" x="-149.86" y="99.06" rot="R180"/>
@@
 <instance part="GND27" gate="1" x="175.26" y="-309.88"/>
 <instance part="R22" gate="G$1" x="238.76" y="-264.16" rot="R90"/>
-<instance part="GND29" gate="1" x="238.76" y="-251.46" rot="MR180"/>
+<instance part="GND29" gate="1" x="238.76" y="-246.38" rot="MR180"/>
 <instance part="P+14" gate="1" x="238.76" y="-276.86" rot="R180"/>
 <instance part="GND28" gate="1" x="-106.68" y="-7.62"/>
@@
 <instance part="R35" gate="G$1" x="-15.24" y="-2.54" rot="R180"/>
 <instance part="GND13" gate="1" x="-17.78" y="-20.32"/>
-<instance part="P+18" gate="1" x="-55.88" y="-22.86" smashed="yes" rot="R180">
-<attribute name="VALUE" x="-55.88" y="-25.4" size="1.778" layer="96"/>
+<instance part="P+18" gate="1" x="-55.88" y="-30.48" smashed="yes" rot="R180">
+<attribute name="VALUE" x="-55.88" y="-33.02" size="1.778" layer="96"/>
 </instance>
 <instance part="P+19" gate="1" x="0" y="-20.32" smashed="yes" rot="R180">
@@
 <instance part="C17" gate="G$1" x="309.88" y="-226.06" rot="R270"/>
 <instance part="GND41" gate="1" x="317.5" y="-226.06" rot="MR270"/>
+<instance part="R19" gate="G$2" x="-165.1" y="142.24"/>
+<instance part="R21" gate="G$2" x="-228.6" y="83.82" rot="R180"/>
+<instance part="R20" gate="G$2" x="-76.2" y="-30.48" rot="R180"/>
+<instance part="R23" gate="G$2" x="165.1" y="-309.88" rot="R180"/>
+<instance part="R22" gate="G$2" x="246.38" y="-246.38"/>
 </instances>
 <busses>
@@
 <pinref part="GND12" gate="1" pin="GND"/>
 <pinref part="R32" gate="G$1" pin="1"/>
+<wire x1="-66.04" y1="-25.4" x2="-66.04" y2="-20.32" width="0.1524" layer="91"/>
+<pinref part="R20" gate="G$2" pin="P$1"/>
 <wire x1="-66.04" y1="-20.32" x2="-66.04" y2="-17.78" width="0.1524" layer="91"/>
+<wire x1="-76.2" y1="-25.4" x2="-76.2" y2="-20.32" width="0.1524" layer="91"/>
+<wire x1="-76.2" y1="-20.32" x2="-66.04" y2="-20.32" width="0.1524" layer="91"/>
+<junction x="-66.04" y="-20.32"/>
 </segment>
 <segment>
@@
 <wire x1="-218.44" y1="114.3" x2="-218.44" y2="111.76" width="0.1524" layer="91"/>
 <pinref part="SAMP_CV" gate="G$1" pin="4"/>
-<wire x1="-218.44" y1="111.76" x2="-218.44" y2="86.36" width="0.1524" layer="91"/>
+<wire x1="-218.44" y1="111.76" x2="-218.44" y2="93.98" width="0.1524" layer="91"/>
+<wire x1="-218.44" y1="93.98" x2="-218.44" y2="86.36" width="0.1524" layer="91"/>
 <wire x1="-223.52" y1="111.76" x2="-218.44" y2="111.76" width="0.1524" layer="91"/>
 <junction x="-218.44" y="111.76"/>
+<pinref part="R21" gate="G$2" pin="P$1"/>
+<wire x1="-228.6" y1="88.9" x2="-228.6" y2="93.98" width="0.1524" layer="91"/>
+<wire x1="-228.6" y1="93.98" x2="-218.44" y2="93.98" width="0.1524" layer="91"/>
+<junction x="-218.44" y="93.98"/>
 </segment>
 <segment>
@@
 <wire x1="175.26" y1="-279.4" x2="175.26" y2="-281.94" width="0.1524" layer="91"/>
 <pinref part="CRUSH_CV" gate="G$1" pin="4"/>
-<wire x1="175.26" y1="-281.94" x2="175.26" y2="-307.34" width="0.1524" layer="91"/>
+<wire x1="175.26" y1="-281.94" x2="175.26" y2="-299.72" width="0.1524" layer="91"/>
+<wire x1="175.26" y1="-299.72" x2="175.26" y2="-307.34" width="0.1524" layer="91"/>
 <wire x1="170.18" y1="-281.94" x2="175.26" y2="-281.94" width="0.1524" layer="91"/>
 <junction x="175.26" y="-281.94"/>
+<pinref part="R23" gate="G$2" pin="P$1"/>
+<wire x1="165.1" y1="-304.8" x2="165.1" y2="-299.72" width="0.1524" layer="91"/>
+<wire x1="165.1" y1="-299.72" x2="175.26" y2="-299.72" width="0.1524" layer="91"/>
+<junction x="175.26" y="-299.72"/>
 </segment>
 <segment>
@@
 <pinref part="GND29" gate="1" pin="GND"/>
 <wire x1="238.76" y1="-256.54" x2="238.76" y2="-254" width="0.1524" layer="91"/>
+<pinref part="R22" gate="G$2" pin="P$1"/>
+<wire x1="238.76" y1="-254" x2="238.76" y2="-248.92" width="0.1524" layer="91"/>
+<wire x1="246.38" y1="-251.46" x2="246.38" y2="-254" width="0.1524" layer="91"/>
+<wire x1="246.38" y1="-254" x2="238.76" y2="-254" width="0.1524" layer="91"/>
+<junction x="238.76" y="-254"/>
 </segment>
 <segment>
@@
 <pinref part="GND21" gate="1" pin="GND"/>
 <wire x1="-149.86" y1="132.08" x2="-149.86" y2="134.62" width="0.1524" layer="91"/>
+<pinref part="R19" gate="G$2" pin="P$1"/>
+<wire x1="-149.86" y1="134.62" x2="-149.86" y2="139.7" width="0.1524" layer="91"/>
+<wire x1="-165.1" y1="137.16" x2="-165.1" y2="134.62" width="0.1524" layer="91"/>
+<wire x1="-165.1" y1="134.62" x2="-149.86" y2="134.62" width="0.1524" layer="91"/>
+<junction x="-149.86" y="134.62"/>
 </segment>
 <segment>
@@
 <segment>
 <pinref part="R33" gate="G$1" pin="1"/>
-<wire x1="-55.88" y1="-20.32" x2="-55.88" y2="-17.78" width="0.1524" layer="91"/>
+<wire x1="-55.88" y1="-27.94" x2="-55.88" y2="-17.78" width="0.1524" layer="91"/>
 <pinref part="P+18" gate="1" pin="+5V"/>
 </segment>

Commit message: v1.3
Parts:
- added C18: 10u, resistor:CPOL-USE2-5
- R17: value 2.7K -> 3.3K
Connections:
- net GND: now also C18.-
- net N$51: now also C18.+
Other:
- moved on the sheet: C8, D1, D2, F2
Changed lines of the file:
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@@
 <?xml version="1.0" encoding="utf-8"?>
 <!DOCTYPE eagle SYSTEM "eagle.dtd">
-<eagle version="6.1">
+<eagle version="6.5.0">
 <drawing>
 <settings>
@@
 <part name="C15" library="resistor" deviceset="CPOL-US" device="E2-5" value="10u"/>
 <part name="GND39" library="supply1" deviceset="GND" device=""/>
-<part name="R17" library="resistor" deviceset="R-US_" device="R0805" value="2.7K"/>
+<part name="R17" library="resistor" deviceset="R-US_" device="R0805" value="3.3K"/>
 <part name="IC1" library="linear" deviceset="TL074" device="D"/>
 <part name="GND4" library="supply1" deviceset="GND" device=""/>
@@
 <part name="C17" library="resistor" deviceset="C-EU" device="C0402" value="0.01uF"/>
 <part name="GND41" library="supply1" deviceset="GND" device=""/>
+<part name="C18" library="resistor" deviceset="CPOL-US" device="E2-5" value="10u"/>
+<part name="GND42" library="supply1" deviceset="GND" device=""/>
 </parts>
 <sheets>
@@
 <instance part="R58" gate="G$1" x="254" y="-294.64" rot="R180"/>
 <instance part="GND7" gate="1" x="266.7" y="-294.64" rot="MR0"/>
-<instance part="GND32" gate="1" x="167.64" y="25.4"/>
-<instance part="P+12" gate="1" x="167.64" y="58.42" smashed="yes">
-<attribute name="VALUE" x="167.64" y="60.96" size="1.778" layer="96" rot="R180"/>
+<instance part="GND32" gate="1" x="175.26" y="25.4"/>
+<instance part="P+12" gate="1" x="175.26" y="58.42" smashed="yes">
+<attribute name="VALUE" x="175.26" y="60.96" size="1.778" layer="96" rot="R180"/>
 </instance>
-<instance part="P+13" gate="1" x="180.34" y="58.42"/>
-<instance part="D1" gate="G$1" x="167.64" y="35.56" rot="R90"/>
+<instance part="P+13" gate="1" x="187.96" y="58.42"/>
+<instance part="D1" gate="G$1" x="175.26" y="35.56" rot="R90"/>
 <instance part="U$2" gate="G$1" x="129.54" y="43.18" rot="R180"/>
-<instance part="C8" gate="G$1" x="193.04" y="40.64"/>
-<instance part="D2" gate="G$1" x="180.34" y="35.56" rot="R90"/>
+<instance part="C8" gate="G$1" x="200.66" y="40.64"/>
+<instance part="D2" gate="G$1" x="187.96" y="35.56" rot="R90"/>
 <instance part="F1" gate="G$1" x="147.32" y="45.72"/>
-<instance part="F2" gate="G$1" x="157.48" y="43.18"/>
+<instance part="F2" gate="G$1" x="167.64" y="43.18"/>
 <instance part="GND33" gate="1" x="147.32" y="25.4"/>
-<instance part="GND34" gate="1" x="180.34" y="25.4"/>
-<instance part="P+16" gate="1" x="193.04" y="58.42" smashed="yes">
-<attribute name="VALUE" x="195.58" y="60.96" size="1.778" layer="96" rot="R180"/>
+<instance part="GND34" gate="1" x="187.96" y="25.4"/>
+<instance part="P+16" gate="1" x="200.66" y="58.42" smashed="yes">
+<attribute name="VALUE" x="203.2" y="60.96" size="1.778" layer="96" rot="R180"/>
 </instance>
-<instance part="GND35" gate="1" x="193.04" y="25.4"/>
+<instance part="GND35" gate="1" x="200.66" y="25.4"/>
 <instance part="F3" gate="G$1" x="111.76" y="33.02"/>
 <instance part="D3" gate="G$1" x="101.6" y="25.4" rot="R270"/>
@@
 <instance part="R23" gate="G$2" x="165.1" y="-309.88" rot="R180"/>
 <instance part="R22" gate="G$2" x="246.38" y="-246.38"/>
+<instance part="C18" gate="G$1" x="157.48" y="35.56"/>
+<instance part="GND42" gate="1" x="157.48" y="25.4"/>
 </instances>
 <busses>
@@
 <segment>
 <pinref part="D1" gate="G$1" pin="A"/>
-<wire x1="167.64" y1="33.02" x2="167.64" y2="27.94" width="0.1524" layer="91"/>
+<wire x1="175.26" y1="33.02" x2="175.26" y2="27.94" width="0.1524" layer="91"/>
 <pinref part="GND32" gate="1" pin="GND"/>
 </segment>
@@
 <segment>
 <pinref part="D2" gate="G$1" pin="A"/>
-<wire x1="180.34" y1="27.94" x2="180.34" y2="33.02" width="0.1524" layer="91"/>
+<wire x1="187.96" y1="27.94" x2="187.96" y2="33.02" width="0.1524" layer="91"/>
 <pinref part="GND34" gate="1" pin="GND"/>
 </segment>
@@
 <pinref part="C8" gate="G$1" pin="-"/>
 <pinref part="GND35" gate="1" pin="GND"/>
-<wire x1="193.04" y1="27.94" x2="193.04" y2="35.56" width="0.1524" layer="91"/>
+<wire x1="200.66" y1="27.94" x2="200.66" y2="35.56" width="0.1524" layer="91"/>
 </segment>
 <segment>
@@
 <pinref part="GND41" gate="1" pin="GND"/>
 <wire x1="312.42" y1="-226.06" x2="314.96" y2="-226.06" width="0.1524" layer="91"/>
+</segment>
+<segment>
+<pinref part="GND42" gate="1" pin="GND"/>
+<pinref part="C18" gate="G$1" pin="-"/>
+<wire x1="157.48" y1="27.94" x2="157.48" y2="30.48" width="0.1524" layer="91"/>
 </segment>
 </net>
@@
 <segment>
 <pinref part="P+13" gate="1" pin="+12V"/>
-<wire x1="180.34" y1="55.88" x2="180.34" y2="43.18" width="0.1524" layer="91"/>
+<wire x1="187.96" y1="55.88" x2="187.96" y2="43.18" width="0.1524" layer="91"/>
 <pinref part="D2" gate="G$1" pin="C"/>
-<wire x1="162.56" y1="43.18" x2="180.34" y2="43.18" width="0.1524" layer="91"/>
-<wire x1="180.34" y1="38.1" x2="180.34" y2="43.18" width="0.1524" layer="91"/>
-<junction x="180.34" y="43.18"/>
+<wire x1="172.72" y1="43.18" x2="187.96" y2="43.18" width="0.1524" layer="91"/>
+<wire x1="187.96" y1="38.1" x2="187.96" y2="43.18" width="0.1524" layer="91"/>
+<junction x="187.96" y="43.18"/>
 <pinref part="F2" gate="G$1" pin="2"/>
 </segment>
@@
 <pinref part="D1" gate="G$1" pin="C"/>
 <pinref part="P+12" gate="1" pin="+5V"/>
-<wire x1="167.64" y1="55.88" x2="167.64" y2="45.72" width="0.1524" layer="91"/>
-<junction x="167.64" y="45.72"/>
+<wire x1="175.26" y1="55.88" x2="175.26" y2="45.72" width="0.1524" layer="91"/>
+<junction x="175.26" y="45.72"/>
 <pinref part="F1" gate="G$1" pin="2"/>
-<wire x1="152.4" y1="45.72" x2="167.64" y2="45.72" width="0.1524" layer="91"/>
-<wire x1="167.64" y1="45.72" x2="167.64" y2="38.1" width="0.1524" layer="91"/>
+<wire x1="152.4" y1="45.72" x2="175.26" y2="45.72" width="0.1524" layer="91"/>
+<wire x1="175.26" y1="45.72" x2="175.26" y2="38.1" width="0.1524" layer="91"/>
 </segment>
 <segment>
 <pinref part="C8" gate="G$1" pin="+"/>
 <pinref part="P+16" gate="1" pin="+5V"/>
-<wire x1="193.04" y1="55.88" x2="193.04" y2="43.18" width="0.1524" layer="91"/>
+<wire x1="200.66" y1="55.88" x2="200.66" y2="43.18" width="0.1524" layer="91"/>
 </segment>
 <segment>
@@
 <segment>
 <pinref part="F2" gate="G$1" pin="1"/>
-<wire x1="137.16" y1="43.18" x2="152.4" y2="43.18" width="0.1524" layer="91"/>
+<wire x1="137.16" y1="43.18" x2="157.48" y2="43.18" width="0.1524" layer="91"/>
 <pinref part="U$2" gate="G$1" pin="9"/>
 <junction x="137.16" y="43.18"/>
+<wire x1="157.48" y1="43.18" x2="162.56" y2="43.18" width="0.1524" layer="91"/>
 <wire x1="121.92" y1="43.18" x2="137.16" y2="43.18" width="0.1524" layer="91"/>
 <pinref part="U$2" gate="G$1" pin="10"/>
-</segment>
-</net>
+<pinref part="C18" gate="G$1" pin="+"/>
+<wire x1="157.48" y1="38.1" x2="157.48" y2="43.18" width="0.1524" layer="91"/>
+<junction x="157.48" y="43.18"/>
+</segment>
+</net>

Commit message: added title and license
Other:
- note added: "Bit Reactor Modular v1.3"
- note added: "Published under the GNU GPL"
- note added: "Rebel Technology 2014"
Changed lines of the file:
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@@
 <?xml version="1.0" encoding="utf-8"?>
 <!DOCTYPE eagle SYSTEM "eagle.dtd">
-<eagle version="6.5.0">
+<eagle version="6.6.0">
 <drawing>
 <settings>
@@
 <text x="185.42" y="-307.34" size="1.778" layer="97" rot="R90">Crush Depth</text>
 <text x="233.68" y="-266.7" size="1.778" layer="97" rot="R90">Crush Level</text>
+<text x="-231.14" y="-271.78" size="12.7" layer="250">Bit Reactor Modular v1.3</text>
+<text x="-231.14" y="-289.56" size="12.7" layer="250">Rebel Technology 2014</text>
+<text x="-231.14" y="-307.34" size="12.7" layer="250">Published under the GNU GPL</text>
 </plain>
 <instances>
