File: ClockDelay/schematics/ClockDelay.sch (EAGLE design)
At the start: 69 parts, among them IC1 TL072P, IC2 MEGA168, Q301 2N3904, Q401 2N3904, Q501 2N3904, Q601 2N3904, Q701 2N3904, Y1 16Mhz

Commit message: turned design upright, fixed board/schematic inconsistency in Y1, fixed DRC errors
Changed lines of the file:
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@@
 <?xml version="1.0" encoding="utf-8"?>
 <!DOCTYPE eagle SYSTEM "eagle.dtd">
-<eagle version="6.3">
+<eagle version="6.6.0">
 <drawing>
 <settings>
@@
 <layers>
 <layer number="1" name="Top" color="4" fill="1" visible="no" active="no"/>
+<layer number="2" name="Route2" color="1" fill="3" visible="no" active="no"/>
+<layer number="3" name="Route3" color="4" fill="3" visible="no" active="no"/>
+<layer number="14" name="Route14" color="1" fill="6" visible="no" active="no"/>
+<layer number="15" name="Route15" color="4" fill="6" visible="no" active="no"/>
 <layer number="16" name="Bottom" color="1" fill="1" visible="no" active="no"/>
 <layer number="17" name="Pads" color="2" fill="1" visible="no" active="no"/>
@@
 <layer number="111" name="LPC17xx" color="7" fill="1" visible="yes" active="yes"/>
 <layer number="112" name="tSilk" color="7" fill="1" visible="yes" active="yes"/>
+<layer number="113" name="Max.sfx.Comments" color="9" fill="1" visible="yes" active="yes"/>
 <layer number="116" name="Patch_BOT" color="7" fill="1" visible="yes" active="yes"/>
 <layer number="121" name="_tsilk" color="7" fill="1" visible="yes" active="yes"/>
@@
 <part name="S1" library="Rebel" deviceset="SWITCH-SPST" device=""/>
 <part name="IC2" library="atmel" deviceset="MEGA8-P" device="" value="MEGA168"/>
-<part name="Y1" library="SparkFun" deviceset="RESONATOR" device="PTH" value="16Mhz"/>
 <part name="P+7" library="supply1" deviceset="+5V" device=""/>
 <part name="C3" library="rcl" deviceset="C-US" device="050-024X044" value="100n"/>
@@
 <part name="P-4" library="supply1" deviceset="-12V" device=""/>
 <part name="JP2" library="SparkFun" deviceset="M04" device="PTH"/>
+<part name="Y1" library="SparkFun" deviceset="RESONATOR" device="PTH" value="16Mhz"/>
 </parts>
 <sheets>
@@
 <instance part="IC1" gate="B" x="71.12" y="-66.04" rot="MR180"/>
 <instance part="IC2" gate="G$1" x="193.04" y="-88.9"/>
-<instance part="Y1" gate="G$1" x="160.02" y="-81.28" rot="R270"/>
 <instance part="P+7" gate="1" x="165.1" y="-50.8"/>
 <instance part="C3" gate="G$1" x="165.1" y="-106.68"/>
@@
 <instance part="P-4" gate="1" x="33.02" y="-81.28"/>
 <instance part="JP2" gate="G$1" x="246.38" y="-68.58" rot="R180"/>
+<instance part="Y1" gate="G$1" x="160.02" y="-81.28" rot="R270"/>
 </instances>
 <busses>
@@
 <pinref part="IC2" gate="G$1" pin="GND@1"/>
 <wire x1="170.18" y1="-91.44" x2="149.86" y2="-91.44" width="0.1524" layer="91"/>
-<pinref part="Y1" gate="G$1" pin="2"/>
-<wire x1="152.4" y1="-81.28" x2="149.86" y2="-81.28" width="0.1524" layer="91"/>
-<wire x1="149.86" y1="-81.28" x2="149.86" y2="-91.44" width="0.1524" layer="91"/>
 <junction x="149.86" y="-91.44"/>
 <pinref part="IC2" gate="G$1" pin="GND"/>
 <wire x1="170.18" y1="-66.04" x2="149.86" y2="-66.04" width="0.1524" layer="91"/>
 <wire x1="149.86" y1="-66.04" x2="149.86" y2="-81.28" width="0.1524" layer="91"/>
+<pinref part="GND9" gate="1" pin="GND"/>
+<wire x1="149.86" y1="-81.28" x2="149.86" y2="-91.44" width="0.1524" layer="91"/>
+<wire x1="149.86" y1="-116.84" x2="149.86" y2="-91.44" width="0.1524" layer="91"/>
+<pinref part="Y1" gate="G$1" pin="2"/>
+<wire x1="149.86" y1="-81.28" x2="152.4" y2="-81.28" width="0.1524" layer="91"/>
 <junction x="149.86" y="-81.28"/>
-<pinref part="GND9" gate="1" pin="GND"/>
-<wire x1="149.86" y1="-116.84" x2="149.86" y2="-91.44" width="0.1524" layer="91"/>
 </segment>
 <segment>
@@
 <segment>
 <pinref part="IC2" gate="G$1" pin="PB6(XTAL1/TOSC1)"/>
+<wire x1="170.18" y1="-78.74" x2="160.02" y2="-78.74" width="0.1524" layer="91"/>
 <pinref part="Y1" gate="G$1" pin="1"/>
-<wire x1="170.18" y1="-78.74" x2="160.02" y2="-78.74" width="0.1524" layer="91"/>
 </segment>
 </net>
@@
 <segment>
 <pinref part="IC2" gate="G$1" pin="PB7(XTAL2/TOSC2)"/>
+<wire x1="170.18" y1="-83.82" x2="160.02" y2="-83.82" width="0.1524" layer="91"/>
 <pinref part="Y1" gate="G$1" pin="3"/>
-<wire x1="170.18" y1="-83.82" x2="160.02" y2="-83.82" width="0.1524" layer="91"/>
-</segment>
-</net>
+</segment>
+</net>

Commit message: added programming header
Parts:
- added JP3: (no value), SparkFun:M06SIP
Connections:
- removed net N$18: IC2.PB4(MISO), LED2.A
- removed net N$19: IC2.PB5(SCK), LED3.A
- removed net N$22: IC2.PB3(MOSI/OC2), LED1.A
- removed net N$39: C1.2, IC2.PC6(/RESET), R1.1
- new net MISO: IC2.PB4(MISO), JP3.3, LED2.A
- new net MOSI: IC2.PB3(MOSI/OC2), JP3.4, LED1.A
- new net RST: C1.2, IC2.PC6(/RESET), JP3.5, R1.1
- new net SCK: IC2.PB5(SCK), JP3.2, LED3.A
- net +5V: now also JP3.6
- net GND: now also JP3.1
