File: PowerBoard/schematics/TransformerBoard.sch (EAGLE design)
At the start: 11 parts

Commit message: rev01
Parts:
- added EARTH: TPPAD1-17, testpad:TPPAD1-17
Connections:
- net +15V: now also U$3G$1.A2, U$5G$1.A2; no longer U$3.A2, U$5.A2
- net -15V: now also U$14G$1.E2, U$4G$1.E2; no longer U$14.E2, U$4.E2
- net E: now also EARTH.TP, U$14G$2.P$1, U$3G$2.P$1, U$4G$2.P$1, U$5G$2.P$1
- net GND: now also U$14G$1.A2, U$3G$1.E2, U$4G$1.A2, U$5G$1.E2; no longer U$14.A2, U$3.E2, U$4.A2, U$5.E2
- net L: now also U$14G$1.A1, U$3G$1.A1, U$4G$1.A1, U$5G$1.A1; no longer U$14.A1, U$3.A1, U$4.A1, U$5.A1
- net N: now also U$14G$1.E1, U$3G$1.E1, U$4G$1.E1, U$5G$1.E1; no longer U$14.E1, U$3.E1, U$4.E1, U$5.E1
Changed lines of the file:
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@@
 <part name="U$14" library="Rebel" deviceset="VTX-214-020" device=""/>
 <part name="SV2" library="con-lstb" deviceset="MA03-1" device=""/>
+<part name="EARTH" library="testpad" deviceset="TP" device="PAD1-17" value="TPPAD1-17"/>
 </parts>
 <sheets>
@@
 <instance part="U$14" gate="G$1" x="0" y="-50.8"/>
 <instance part="SV2" gate="G$1" x="68.58" y="-2.54" rot="R180"/>
+<instance part="EARTH" gate="G$1" x="-20.32" y="17.78"/>
+<instance part="U$3" gate="G$2" x="38.1" y="55.88"/>
+<instance part="U$5" gate="G$2" x="50.8" y="55.88"/>
+<instance part="U$4" gate="G$2" x="60.96" y="55.88"/>
+<instance part="U$14" gate="G$2" x="71.12" y="55.88"/>
 </instances>
 <busses>
@@
 <segment>
 <pinref part="X1" gate="-2" pin="S"/>
-<wire x1="-30.48" y1="10.16" x2="-22.86" y2="10.16" width="0.1524" layer="91"/>
+<wire x1="-30.48" y1="10.16" x2="-20.32" y2="10.16" width="0.1524" layer="91"/>
 <label x="-27.94" y="10.16" size="1.778" layer="95"/>
-</segment>
-</net>
+<pinref part="EARTH" gate="G$1" pin="TP"/>
+<wire x1="-20.32" y1="10.16" x2="-20.32" y2="15.24" width="0.1524" layer="91"/>
+</segment>
+<segment>
+<pinref part="U$3" gate="G$2" pin="P$1"/>
+<wire x1="27.94" y1="48.26" x2="38.1" y2="48.26" width="0.1524" layer="91"/>
+<wire x1="38.1" y1="48.26" x2="38.1" y2="50.8" width="0.1524" layer="91"/>
+<label x="30.48" y="48.26" size="1.778" layer="95"/>
+<pinref part="U$5" gate="G$2" pin="P$1"/>
+<wire x1="38.1" y1="48.26" x2="50.8" y2="48.26" width="0.1524" layer="91"/>
+<wire x1="50.8" y1="48.26" x2="50.8" y2="50.8" width="0.1524" layer="91"/>
+<junction x="38.1" y="48.26"/>
+<pinref part="U$4" gate="G$2" pin="P$1"/>
+<wire x1="50.8" y1="48.26" x2="60.96" y2="48.26" width="0.1524" layer="91"/>
+<wire x1="60.96" y1="48.26" x2="60.96" y2="50.8" width="0.1524" layer="91"/>
+<junction x="50.8" y="48.26"/>
+<pinref part="U$14" gate="G$2" pin="P$1"/>
+<wire x1="60.96" y1="48.26" x2="71.12" y2="48.26" width="0.1524" layer="91"/>
+<wire x1="71.12" y1="48.26" x2="71.12" y2="50.8" width="0.1524" layer="91"/>
+<junction x="60.96" y="48.26"/>
+</segment>
+</net>
