File: PowerBoard/schematics/PowerBoard.brd (EAGLE design)
At the start: 139.7 x 44.1 mm, 65 parts, among them IC100 LM317MABDT, IC200 LM317MABDT, IC300 337, X1 22-27-2031-03, X2 22-27-2031-03, X3 22-27-2031-03, X4 22-27-2031-03

Commit message: changed capacitor values - only use 10uF 1206 and 100nF 0603 ceramic film
Parts:
- C101, C104, C201, C204, C302, C304: value 10u -> dnp
- C103, C203, C303: value 1u -> 100n
- C106, C107, C206, C207, C306, C307: value (none) -> 10u
- R1, R3: value 1k -> 2k
- R102, R302: value 2k -> 1k91
Changed lines of the file:
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@@
 <attribute name="NAME" x="87.63" y="10.922" size="1.016" layer="25" font="vector" align="bottom-center"/>
 </element>
-<element name="R102" library="Rebel" package="0603" value="2k" x="21.59" y="13.97" smashed="yes">
+<element name="R102" library="Rebel" package="0603" value="1k91" x="21.59" y="13.97" smashed="yes">
 <attribute name="NAME" x="21.59" y="14.732" size="1.016" layer="25" font="vector" align="bottom-center"/>
 </element>
@@
 <attribute name="NAME" x="54.61" y="15.748" size="1.016" layer="25" font="vector" rot="R180" align="bottom-center"/>
 </element>
-<element name="R302" library="Rebel" package="0603" value="2k" x="87.63" y="13.97" smashed="yes" rot="R180">
+<element name="R302" library="Rebel" package="0603" value="1k91" x="87.63" y="13.97" smashed="yes" rot="R180">
 <attribute name="NAME" x="87.63" y="14.732" size="1.016" layer="25" font="vector" align="bottom-center"/>
 </element>
-<element name="C302" library="rcl" package="153CLV-0810" value="10u" x="87.63" y="27.94" smashed="yes" rot="R90">
+<element name="C302" library="rcl" package="153CLV-0810" value="dnp" x="87.63" y="27.94" smashed="yes" rot="R90">
 <attribute name="NAME" x="93.26" y="25.555" size="1.27" layer="25" rot="R90"/>
 <attribute name="VALUE" x="93.415" y="23.615" size="1.27" layer="27" rot="R90"/>
 </element>
-<element name="C104" library="rcl" package="153CLV-0810" value="10u" x="21.59" y="27.94" smashed="yes" rot="R270">
+<element name="C104" library="rcl" package="153CLV-0810" value="dnp" x="21.59" y="27.94" smashed="yes" rot="R270">
 <attribute name="NAME" x="27.22" y="25.555" size="1.27" layer="25" rot="R90"/>
 <attribute name="VALUE" x="15.805" y="32.265" size="1.27" layer="27" rot="R270"/>
 </element>
-<element name="C204" library="rcl" package="153CLV-0810" value="10u" x="54.61" y="27.94" smashed="yes" rot="R270">
+<element name="C204" library="rcl" package="153CLV-0810" value="dnp" x="54.61" y="27.94" smashed="yes" rot="R270">
 <attribute name="NAME" x="60.24" y="25.555" size="1.27" layer="25" rot="R90"/>
 <attribute name="VALUE" x="48.825" y="32.265" size="1.27" layer="27" rot="R270"/>
 </element>
-<element name="C304" library="rcl" package="153CLV-0810" value="10u" x="100.33" y="27.94" smashed="yes" rot="R90">
+<element name="C304" library="rcl" package="153CLV-0810" value="dnp" x="100.33" y="27.94" smashed="yes" rot="R90">
 <attribute name="NAME" x="105.96" y="25.555" size="1.27" layer="25" rot="R90"/>
 <attribute name="VALUE" x="106.115" y="23.615" size="1.27" layer="27" rot="R90"/>
@@
 <attribute name="VALUE" x="95.25" y="8.89" size="1.27" layer="27" rot="R180"/>
 </element>
-<element name="R1" library="Rebel" package="0603" value="1k" x="33.02" y="6.35" smashed="yes" rot="R180">
+<element name="R1" library="Rebel" package="0603" value="2k" x="33.02" y="6.35" smashed="yes" rot="R180">
 <attribute name="NAME" x="33.02" y="8.128" size="1.016" layer="25" font="vector" rot="R180" align="bottom-center"/>
 </element>
@@
 <attribute name="NAME" x="66.04" y="8.128" size="1.016" layer="25" font="vector" rot="R180" align="bottom-center"/>
 </element>
-<element name="R3" library="Rebel" package="0603" value="1k" x="88.9" y="6.35" smashed="yes">
+<element name="R3" library="Rebel" package="0603" value="2k" x="88.9" y="6.35" smashed="yes">
 <attribute name="NAME" x="88.9" y="4.572" size="1.016" layer="25" font="vector" align="bottom-center"/>
 </element>
-<element name="C103" library="rcl" package="C0603" value="1u" x="38.735" y="13.97" smashed="yes" rot="R180">
+<element name="C103" library="rcl" package="C0603" value="100n" x="38.735" y="13.97" smashed="yes" rot="R180">
 <attribute name="NAME" x="37.465" y="14.605" size="1.016" layer="25"/>
 <attribute name="VALUE" x="39.37" y="15.875" size="1.27" layer="27" rot="R180"/>
 </element>
-<element name="C203" library="rcl" package="C0603" value="1u" x="71.755" y="13.97" smashed="yes" rot="R180">
+<element name="C203" library="rcl" package="C0603" value="100n" x="71.755" y="13.97" smashed="yes" rot="R180">
 <attribute name="NAME" x="70.485" y="14.605" size="1.016" layer="25"/>
 <attribute name="VALUE" x="72.39" y="15.875" size="1.27" layer="27" rot="R180"/>
@@
 <attribute name="VALUE" x="69.596" y="8.509" size="0.4064" layer="27" rot="R180"/>
 </element>
-<element name="C101" library="rcl" package="153CLV-0810" value="10u" x="34.29" y="27.94" smashed="yes" rot="R270">
+<element name="C101" library="rcl" package="153CLV-0810" value="dnp" x="34.29" y="27.94" smashed="yes" rot="R270">
 <attribute name="NAME" x="39.92" y="25.555" size="1.27" layer="25" rot="R90"/>
 <attribute name="VALUE" x="28.505" y="32.265" size="1.27" layer="27" rot="R270"/>
 </element>
-<element name="C201" library="rcl" package="153CLV-0810" value="10u" x="67.31" y="27.94" smashed="yes" rot="R270">
+<element name="C201" library="rcl" package="153CLV-0810" value="dnp" x="67.31" y="27.94" smashed="yes" rot="R270">
 <attribute name="NAME" x="72.94" y="25.555" size="1.27" layer="25" rot="R90"/>
 <attribute name="VALUE" x="61.525" y="32.265" size="1.27" layer="27" rot="R270"/>
@@
 <attribute name="VALUE" x="86.995" y="14.605" size="1.27" layer="27"/>
 </element>
-<element name="C303" library="rcl" package="C0603" value="1u" x="101.6" y="13.97" smashed="yes" rot="R180">
+<element name="C303" library="rcl" package="C0603" value="100n" x="101.6" y="13.97" smashed="yes" rot="R180">
 <attribute name="NAME" x="100.33" y="14.605" size="1.016" layer="25"/>
 <attribute name="VALUE" x="102.235" y="15.875" size="1.27" layer="27" rot="R180"/>
@@
 <attribute name="VALUE" x="115.5969" y="36.0411" size="0.8128" layer="27" ratio="10"/>
 </element>
-<element name="C106" library="rcl" package="C1206" value="" x="36.195" y="17.145" smashed="yes">
+<element name="C106" library="rcl" package="C1206" value="10u" x="36.195" y="17.145" smashed="yes">
 <attribute name="NAME" x="35.56" y="18.415" size="1.27" layer="25"/>
 <attribute name="VALUE" x="34.925" y="14.605" size="1.27" layer="27"/>
 </element>
-<element name="C206" library="rcl" package="C1206" value="" x="69.215" y="17.145" smashed="yes">
+<element name="C206" library="rcl" package="C1206" value="10u" x="69.215" y="17.145" smashed="yes">
 <attribute name="NAME" x="68.58" y="18.415" size="1.27" layer="25"/>
 <attribute name="VALUE" x="67.945" y="14.605" size="1.27" layer="27"/>
 </element>
-<element name="C207" library="rcl" package="C1206" value="" x="69.215" y="20.955" smashed="yes">
+<element name="C207" library="rcl" package="C1206" value="10u" x="69.215" y="20.955" smashed="yes">
 <attribute name="NAME" x="68.58" y="22.225" size="1.27" layer="25"/>
 <attribute name="VALUE" x="67.945" y="18.415" size="1.27" layer="27"/>
 </element>
-<element name="C107" library="rcl" package="C1206" value="" x="36.195" y="20.955" smashed="yes">
+<element name="C107" library="rcl" package="C1206" value="10u" x="36.195" y="20.955" smashed="yes">
 <attribute name="NAME" x="35.56" y="22.225" size="1.27" layer="25"/>
 <attribute name="VALUE" x="34.925" y="18.415" size="1.27" layer="27"/>
 </element>
-<element name="C307" library="rcl" package="C1206" value="" x="87.63" y="19.685" smashed="yes">
+<element name="C307" library="rcl" package="C1206" value="10u" x="87.63" y="19.685" smashed="yes">
 <attribute name="NAME" x="85.725" y="20.955" size="1.27" layer="25"/>
 <attribute name="VALUE" x="86.36" y="17.145" size="1.27" layer="27"/>
 </element>
-<element name="C306" library="rcl" package="C1206" value="" x="101.6" y="20.955" smashed="yes">
+<element name="C306" library="rcl" package="C1206" value="10u" x="101.6" y="20.955" smashed="yes">
 <attribute name="NAME" x="101.6" y="22.225" size="1.27" layer="25"/>
 <attribute name="VALUE" x="100.33" y="18.415" size="1.27" layer="27"/>
