File: OWL/schematics/owl-digital.brd (EAGLE design)
At the start: 59.6 x 55.9 mm, 70 parts, among them IC1 TLV1117-33CDCY, IC3 IS61WV51216BLL-10TLI, Q1 12.288MHz, Q2 8MHz, U2 WM8731, U4 STM32F405ZGT6

Commit message: tons of old updates in one fat commit
Connections:
- net UART_RX renamed PB6
- net UART_TX renamed PB7
Changed lines of the file:
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@@
 <text x="3.4925" y="44.1325" size="0.8128" layer="21" font="vector" rot="SR90">PE5</text>
 <text x="3.4925" y="21.1582" size="0.8128" layer="21" font="vector" rot="SR90">PF9</text>
-<text x="10.4775" y="53.0225" size="0.8128" layer="21" font="vector" rot="SR0">PB6</text>
-<text x="13.0175" y="53.0225" size="0.8128" layer="21" font="vector" rot="SR0">PB7</text>
+<text x="13.0175" y="53.0225" size="0.8128" layer="21" font="vector" rot="SR0">PB6</text>
+<text x="10.4775" y="53.0225" size="0.8128" layer="21" font="vector" rot="SR0">PB7</text>
 <text x="16.1925" y="53.6575" size="0.8128" layer="21" font="vector" rot="SR270">BOOT0</text>
 <text x="18.7325" y="53.6575" size="0.8128" layer="21" font="vector" rot="SR270">PG14</text>
@@
 <contactref element="U4" pad="135"/>
 </signal>
-<signal name="UART_RX">
+<signal name="PB6">
 <contactref element="U4" pad="136"/>
 <wire x1="13.0302" y1="47.5488" x2="13.0302" y2="46.3423" width="0.2032" layer="1"/>
@@
 <wire x1="13.335" y1="54.61" x2="13.97" y2="55.245" width="0.2032" layer="16"/>
 </signal>
-<signal name="UART_TX">
+<signal name="PB7">
 <contactref element="U4" pad="137"/>
 <wire x1="12.5222" y1="47.5488" x2="12.5222" y2="46.4947" width="0.2032" layer="1"/>

Commit message: updated to rev06
Parts:
- C302, C308: value 1u -> 4u7
Other:
- board text added: "OWL Rev06"
- board text removed: "OWL Rev05"
Changed lines of the file:
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@@
 <?xml version="1.0" encoding="utf-8"?>
 <!DOCTYPE eagle SYSTEM "eagle.dtd">
-<eagle version="6.5.0">
+<eagle version="7.5.0">
 <drawing>
 <settings>
@@
 <text x="13.97" y="14.605" size="0.8128" layer="21" font="vector" rot="SR0">PB1</text>
 <text x="13.97" y="15.5575" size="0.8128" layer="21" font="vector" rot="SR0">PB2</text>
-<text x="21.59" y="18.7325" size="1.9304" layer="21" font="vector">OWL Rev05</text>
+<text x="21.59" y="18.7325" size="1.9304" layer="21" font="vector">OWL Rev06</text>
 <text x="26.035" y="1.27" size="1.016" layer="21" font="vector" rot="SR0">5v</text>
 <text x="2.8575" y="4.445" size="1.016" layer="21" font="vector" rot="SR0" align="center-left">gnd</text>
@@
 <dimension x1="1.27" y1="55.245" x2="49.53" y2="55.245" x3="25.4" y3="58.42" textsize="1.778" layer="47" unit="mil"/>
 <text x="51.1175" y="54.9275" size="0.8128" layer="21" font="vector" rot="SR0">gnd</text>
+<text x="51.435" y="38.4175" size="1.9304" layer="22" font="vector" rot="MR270">OWL Rev06</text>
+<text x="52.4721375" y="17.0357375" size="1.9304" layer="22" font="vector" rot="MR90">Rebel Technology</text>
 </plain>
 <attributes>
@@
 <pass name="Default">
 <param name="RoutingGrid" value="10mil"/>
+<param name="AutoGrid" value="1"/>
+<param name="Efforts" value="0"/>
+<param name="TopRouterVariant" value="1"/>
 <param name="tpViaShape" value="round"/>
 <param name="PrefDir.1" value="|"/>
@@
 <attribute name="VALUE" x="35.179" y="14.732" size="1.27" layer="27" rot="R180"/>
 </element>
-<element name="C308" library="resistor" package="C1206" value="1u" x="49.53" y="6.0325" smashed="yes">
+<element name="C308" library="resistor" package="C1206" value="4u7" x="49.53" y="6.0325" smashed="yes">
 <attribute name="NAME" x="47.3075" y="7.1755" size="1.27" layer="25"/>
 <attribute name="VALUE" x="48.26" y="3.6195" size="1.27" layer="27"/>
@@
 <attribute name="VALUE" x="34.544" y="6.1595" size="1.27" layer="27" rot="R180"/>
 </element>
-<element name="C302" library="resistor" package="C1206" value="1u" x="30.1625" y="5.715" smashed="yes" rot="R270">
+<element name="C302" library="resistor" package="C1206" value="4u7" x="30.1625" y="5.715" smashed="yes" rot="R270">
 <attribute name="NAME" x="29.0195" y="3.4925" size="1.27" layer="25" rot="R90"/>
 <attribute name="VALUE" x="27.7495" y="6.985" size="1.27" layer="27" rot="R270"/>
