File: OWL/schematics/owl-digital-2.sch (EAGLE design)
At the start: 72 parts, among them IC1 LMC6482, IC10 IS42S16400J, IC4 CS4271, IC8 STM32F756ZLQFP144, IC9 N25Q128A13, U4 V_REG_LM3940IMP, Y1 24.576MHz, Y3 25MHz

Commit message: changed some labels
Connections:
- net CS_VQ1: now also IC1A.+IN
Other:
- moved on the sheet: C3
Changed lines of the file:
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@@
 <instance part="IC1" gate="B" x="401.32" y="0"/>
 <instance part="IC1" gate="P" x="401.32" y="25.4"/>
-<instance part="GND4" gate="1" x="401.32" y="12.7"/>
+<instance part="GND4" gate="1" x="401.32" y="10.16"/>
 <instance part="P+4" gate="1" x="401.32" y="38.1"/>
 <instance part="C1" gate="G$1" x="383.54" y="22.86"/>
 <instance part="C2" gate="G$1" x="373.38" y="22.86"/>
-<instance part="GND5" gate="1" x="383.54" y="12.7"/>
-<instance part="GND7" gate="1" x="373.38" y="12.7"/>
-<instance part="GND8" gate="1" x="388.62" y="-7.62"/>
-<instance part="C3" gate="G$1" x="431.8" y="22.86"/>
-<instance part="GND9" gate="1" x="431.8" y="12.7"/>
-<instance part="P+7" gate="1" x="431.8" y="30.48"/>
+<instance part="GND5" gate="1" x="383.54" y="10.16"/>
+<instance part="GND7" gate="1" x="373.38" y="10.16"/>
+<instance part="GND8" gate="1" x="388.62" y="-15.24"/>
+<instance part="C3" gate="G$1" x="431.8" y="25.4"/>
+<instance part="GND9" gate="1" x="431.8" y="10.16"/>
+<instance part="P+7" gate="1" x="431.8" y="38.1"/>
 </instances>
 <busses>
@@
 <pinref part="IC1" gate="P" pin="V-"/>
 <pinref part="GND4" gate="1" pin="GND"/>
-<wire x1="401.32" y1="15.24" x2="401.32" y2="17.78" width="0.1524" layer="91"/>
+<wire x1="401.32" y1="12.7" x2="401.32" y2="17.78" width="0.1524" layer="91"/>
 </segment>
 <segment>
 <pinref part="GND7" gate="1" pin="GND"/>
 <pinref part="C2" gate="G$1" pin="2"/>
-<wire x1="373.38" y1="15.24" x2="373.38" y2="17.78" width="0.1524" layer="91"/>
+<wire x1="373.38" y1="12.7" x2="373.38" y2="17.78" width="0.1524" layer="91"/>
 </segment>
 <segment>
 <pinref part="GND5" gate="1" pin="GND"/>
 <pinref part="C1" gate="G$1" pin="2"/>
-<wire x1="383.54" y1="15.24" x2="383.54" y2="17.78" width="0.1524" layer="91"/>
+<wire x1="383.54" y1="12.7" x2="383.54" y2="17.78" width="0.1524" layer="91"/>
 </segment>
 <segment>
 <pinref part="GND8" gate="1" pin="GND"/>
-<wire x1="388.62" y1="-5.08" x2="388.62" y2="2.54" width="0.1524" layer="91"/>
+<wire x1="388.62" y1="-12.7" x2="388.62" y2="2.54" width="0.1524" layer="91"/>
 <pinref part="IC1" gate="B" pin="+IN"/>
 <wire x1="388.62" y1="2.54" x2="393.7" y2="2.54" width="0.1524" layer="91"/>
@@
 <pinref part="GND9" gate="1" pin="GND"/>
 <pinref part="C3" gate="G$1" pin="2"/>
-<wire x1="431.8" y1="15.24" x2="431.8" y2="17.78" width="0.1524" layer="91"/>
+<wire x1="431.8" y1="12.7" x2="431.8" y2="20.32" width="0.1524" layer="91"/>
 </segment>
 </net>
@@
 <pinref part="C3" gate="G$1" pin="1"/>
 <pinref part="P+7" gate="1" pin="+5V"/>
-<wire x1="431.8" y1="25.4" x2="431.8" y2="27.94" width="0.1524" layer="91"/>
+<wire x1="431.8" y1="27.94" x2="431.8" y2="35.56" width="0.1524" layer="91"/>
 </segment>
 </net>
@@
 <label x="363.22" y="27.94" size="1.778" layer="95"/>
 <junction x="373.38" y="27.94"/>
+<pinref part="IC1" gate="A" pin="+IN"/>
 </segment>
 </net>
@@
 <pinref part="IC1" gate="A" pin="-IN"/>
 <wire x1="393.7" y1="22.86" x2="391.16" y2="22.86" width="0.1524" layer="91"/>
-<wire x1="391.16" y1="22.86" x2="391.16" y2="20.32" width="0.1524" layer="91"/>
+<wire x1="391.16" y1="22.86" x2="391.16" y2="15.24" width="0.1524" layer="91"/>
 <pinref part="IC1" gate="A" pin="OUT"/>
-<wire x1="391.16" y1="20.32" x2="411.48" y2="20.32" width="0.1524" layer="91"/>
-<wire x1="411.48" y1="20.32" x2="411.48" y2="25.4" width="0.1524" layer="91"/>
+<wire x1="391.16" y1="15.24" x2="411.48" y2="15.24" width="0.1524" layer="91"/>
+<wire x1="411.48" y1="15.24" x2="411.48" y2="25.4" width="0.1524" layer="91"/>
 <wire x1="411.48" y1="25.4" x2="408.94" y2="25.4" width="0.1524" layer="91"/>
 <label x="411.48" y="25.4" size="1.778" layer="95"/>
@@
 <pinref part="IC1" gate="B" pin="-IN"/>
 <wire x1="393.7" y1="-2.54" x2="391.16" y2="-2.54" width="0.1524" layer="91"/>
-<wire x1="391.16" y1="-2.54" x2="391.16" y2="-5.08" width="0.1524" layer="91"/>
-<wire x1="391.16" y1="-5.08" x2="411.48" y2="-5.08" width="0.1524" layer="91"/>
-<wire x1="411.48" y1="-5.08" x2="411.48" y2="0" width="0.1524" layer="91"/>
+<wire x1="391.16" y1="-2.54" x2="391.16" y2="-10.16" width="0.1524" layer="91"/>
+<wire x1="391.16" y1="-10.16" x2="411.48" y2="-10.16" width="0.1524" layer="91"/>
+<wire x1="411.48" y1="-10.16" x2="411.48" y2="0" width="0.1524" layer="91"/>
 <pinref part="IC1" gate="B" pin="OUT"/>
 <wire x1="411.48" y1="0" x2="408.94" y2="0" width="0.1524" layer="91"/>
