File: OWL 2/schematic/owl-digital-2.sch (EAGLE design)
At the start: 72 parts, among them IC1 LMC6482, IC10 IS42S16400J, IC4 CS4271, IC8 STM32F756ZLQFP144, IC9 N25Q128A13, U4 V_REG_LM3940IMP, Y1 24.576MHz, Y3 25MHz

Commit message: Code to run SDRAM working
Connections:
- removed net TOP_GP5: JP4.3
- net +3V3: now also JP4.1
- net GND: now also JP4.3
Changed lines of the file:
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@@
 <?xml version="1.0" encoding="utf-8"?>
 <!DOCTYPE eagle SYSTEM "eagle.dtd">
-<eagle version="7.5.0">
+<eagle version="6.6.0">
 <drawing>
 <settings>
@@
 <part name="GND9" library="supply1" deviceset="GND" device=""/>
 <part name="P+7" library="supply1" deviceset="+5V" device=""/>
+<part name="+3V15" library="supply1" deviceset="+3V3" device=""/>
+<part name="GND12" library="supply1" deviceset="GND" device=""/>
 </parts>
 <sheets>
@@
 <instance part="GND9" gate="1" x="431.8" y="10.16"/>
 <instance part="P+7" gate="1" x="431.8" y="38.1"/>
+<instance part="+3V15" gate="G$1" x="259.08" y="17.78" rot="R180"/>
+<instance part="GND12" gate="1" x="254" y="17.78"/>
 </instances>
 <busses>
@@
 <wire x1="431.8" y1="12.7" x2="431.8" y2="20.32" width="0.1524" layer="91"/>
 </segment>
+<segment>
+<pinref part="GND12" gate="1" pin="GND"/>
+<pinref part="JP4" gate="G$1" pin="3"/>
+<wire x1="254" y1="20.32" x2="254" y2="30.48" width="0.1524" layer="91"/>
+</segment>
 </net>
 <net name="FLASH_NCS" class="0">
@@
 <wire x1="106.68" y1="-45.72" x2="106.68" y2="-43.18" width="0.1524" layer="91"/>
 </segment>
+<segment>
+<pinref part="+3V15" gate="G$1" pin="+3V3"/>
+<pinref part="JP4" gate="G$1" pin="1"/>
+<wire x1="259.08" y1="20.32" x2="259.08" y2="30.48" width="0.1524" layer="91"/>
+</segment>
 </net>
 <net name="ADC4" class="0">
@@
 </segment>
 </net>
-<net name="TOP_GP5" class="0">
-<segment>
-<pinref part="JP4" gate="G$1" pin="3"/>
-<wire x1="254" y1="30.48" x2="254" y2="17.78" width="0.1524" layer="91"/>
-<label x="254" y="17.78" size="1.778" layer="95" rot="R90"/>
-</segment>
-</net>
