File: Expander/schematics/Expander.brd (EAGLE design)
At the start: 61.1 x 100 mm, 127 parts, among them P1 THONKICONN, P10 THONKICONN, P11 THONKICONN, P12 THONKICONN, P13 THONKICONN, P14 THONKICONN, P15 THONKICONN, P16 THONKICONN, P2 THONKICONN, P3 THONKICONN, P4 THONKICONN, P5 THONKICONN, P6 THONKICONN, P7 THONKICONN, P8 THONKICONN, P9 THONKICONN, U1 MAX11300GTLTQFP, U2 STM32F100CBT6B, U3 TLC5946, U4 LM317, U5 NCP702, X2 53048-05, X3 53047-02, Y2 8MHz

Commit message: renamed temperature nets
Connections:
- net N$10 renamed D0N
- net N$9 renamed D0P
Changed lines of the file:
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@@
 <wire x1="19.05" y1="66.675" x2="17.78" y2="65.405" width="0.4064" layer="1"/>
 </signal>
-<signal name="N$9">
+<signal name="D0P">
 <contactref element="U1" pad="13"/>
 <contactref element="X3" pad="1"/>
@@
 <wire x1="49.74" y1="39.013615625" x2="50.44749375" y2="39.721109375" width="0.254" layer="1"/>
 </signal>
-<signal name="N$10">
+<signal name="D0N">
 <contactref element="U1" pad="14"/>
 <contactref element="X3" pad="2"/>

Commit message: updated Expander drawings and designs
Parts:
- added T1: 2N3904, transistor:TO92
Connections:
- net D0N: now also T1.3
- net D0P: now also T1.1, T1.2
Changed lines of the file:
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@@
 </element>
 <element name="CN1" library="Rebel" package="JST-B3B-PH-KL" value="" x="59.055" y="56.515" smashed="yes" rot="MR270"/>
+<element name="T1" library="transistor" package="TO92" value="2N3904" x="-2.54" y="-4.445"/>
 </elements>
 <signals>
@@
 <wire x1="49.74" y1="38.54" x2="49.74" y2="39.013615625" width="0.254" layer="1"/>
 <wire x1="49.74" y1="39.013615625" x2="50.44749375" y2="39.721109375" width="0.254" layer="1"/>
+<contactref element="T1" pad="2"/>
+<contactref element="T1" pad="1"/>
+<wire x1="-2.54" y1="-2.54" x2="49.74" y2="38.54" width="0" layer="19" extent="1-1"/>
+<wire x1="-1.27" y1="-4.445" x2="-2.54" y2="-2.54" width="0" layer="19" extent="1-1"/>
 </signal>
 <signal name="D0N">
@@
 <wire x1="49.24" y1="38.54" x2="49.24" y2="40.281378125" width="0.254" layer="1"/>
 <wire x1="49.24" y1="40.281378125" x2="49.5636125" y2="40.604990625" width="0.254" layer="1"/>
+<contactref element="T1" pad="3"/>
+<wire x1="-3.81" y1="-4.445" x2="49.24" y2="38.54" width="0" layer="19" extent="1-1"/>
 </signal>
 <signal name="N$16">

Commit message: changes from Nov/Dec
Parts:
- added C32, C33, C34: 4u7, Rebel:C0603
Connections:
- new net N$2: C34.1, U1.10
- new net N$4: C33.1, U1.11
- new net N$5: C32.1, U1.12
- net GND: now also C32.2, C33.2, C34.2
Changed lines of the file:
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@@
 <element name="CN1" library="Rebel" package="JST-B3B-PH-KL" value="" x="59.055" y="56.515" smashed="yes" rot="MR270"/>
 <element name="T1" library="transistor" package="TO92" value="2N3904" x="-2.54" y="-4.445"/>
+<element name="C32" library="Rebel" package="C0603" value="4u7" x="-2.54" y="-8.89"/>
+<element name="C33" library="Rebel" package="C0603" value="4u7" x="-2.54" y="-12.065"/>
+<element name="C34" library="Rebel" package="C0603" value="4u7" x="-2.54" y="-15.24"/>
 </elements>
 <signals>
@@
 <wire x1="42.79" y1="5.7875" x2="42.8625" y2="5.715" width="0.4064" layer="1"/>
 <via x="42.8625" y="5.715" extent="1-16" drill="0.5"/>
+<contactref element="C34" pad="2"/>
+<contactref element="C33" pad="2"/>
+<contactref element="C32" pad="2"/>
+<wire x1="56.8325" y1="75.565" x2="56.73" y2="79.375" width="0" layer="19" extent="1-1"/>
+<wire x1="58" y1="71.755" x2="56.73" y2="74.295" width="0" layer="19" extent="1-1"/>
+<wire x1="52.07" y1="74.295" x2="56.73" y2="74.295" width="0" layer="19" extent="1-1"/>
+<wire x1="46.775" y1="74.93" x2="51.65" y2="74.93" width="0" layer="19" extent="1-1"/>
+<wire x1="45.085" y1="73.66" x2="46.0375" y2="74.93" width="0" layer="19" extent="1-1"/>
+<wire x1="47.625" y1="81.5975" x2="46.775" y2="74.93" width="0" layer="19" extent="1-1"/>
+<wire x1="37.25" y1="74.295" x2="44.069" y2="73.2028" width="0" layer="19" extent="1-1"/>
+<wire x1="37.25" y1="71.755" x2="37.25" y2="74.295" width="0" layer="19" extent="1-1"/>
+<wire x1="37.25" y1="79.375" x2="36.98875" y2="75.565" width="0" layer="19" extent="1-1"/>
+<wire x1="44.92625" y1="63.1825" x2="44.6278" y2="73.2028" width="0" layer="19" extent="1-1"/>
+<wire x1="51.27625" y1="63.1825" x2="51.22" y2="63.12625" width="0" layer="19" extent="1-1"/>
+<wire x1="44.9825" y1="59.905" x2="44.92625" y2="63.1825" width="0" layer="19" extent="1-1"/>
+<wire x1="43.815" y1="58.57875" x2="44.7675" y2="59.69" width="0" layer="19" extent="1-1"/>
+<wire x1="43.18" y1="58.635" x2="43.33875" y2="58.57875" width="0" layer="19" extent="1-1"/>
+<wire x1="41.5925" y1="56.515" x2="42.2275" y2="58.57875" width="0" layer="19" extent="1-1"/>
+<wire x1="34.925" y1="53.975" x2="34.925" y2="56.515" width="0" layer="19" extent="1-1"/>
+<wire x1="35.40125" y1="60.16625" x2="34.925" y2="56.515" width="0" layer="19" extent="1-1"/>
+<wire x1="44.45" y1="51.435" x2="44.7294" y2="56.2864" width="0" layer="19" extent="1-1"/>
+<wire x1="42.8625" y1="48.5775" x2="42.7736" y2="51.308" width="0" layer="19" extent="1-1"/>
+<wire x1="42.8625" y1="44.5525" x2="42.8625" y2="47.9425" width="0" layer="19" extent="1-1"/>
+<wire x1="42.6475" y1="44.5525" x2="42.8625" y2="44.5525" width="0" layer="19" extent="1-1"/>
+<wire x1="45.72" y1="41.91" x2="43.4975" y2="44.1325" width="0" layer="19" extent="1-1"/>
+<wire x1="47.24" y1="38.54" x2="46.4575" y2="41.91" width="0" layer="19" extent="1-1"/>
+<wire x1="49.2125" y1="32.0675" x2="49.24" y2="32.04" width="0" layer="19" extent="1-1"/>
+<wire x1="44.7675" y1="32.0675" x2="44.74" y2="32.04" width="0" layer="19" extent="1-1"/>
+<wire x1="52.64875" y1="31.2175" x2="51.24" y2="32.04" width="0" layer="19" extent="1-1"/>
+<wire x1="46.99" y1="36.5125" x2="47.74" y2="35.04" width="0" layer="19" extent="1-1"/>
+<wire x1="49.2125" y1="34.29" x2="47.74" y2="35.04" width="0" layer="19" extent="1-1"/>
+<wire x1="49.2125" y1="36.5125" x2="47.74" y2="35.04" width="0" layer="19" extent="1-1"/>
+<wire x1="50.4825" y1="37.7825" x2="49.2125" y2="36.5125" width="0" layer="19" extent="1-1"/>
+<wire x1="44.7675" y1="36.5125" x2="46.99" y2="36.5125" width="0" layer="19" extent="1-1"/>
+<wire x1="46.99" y1="32.0675" x2="46.99" y2="34.29" width="0" layer="19" extent="1-1"/>
+<wire x1="44.7675" y1="34.29" x2="46.99" y2="34.29" width="0" layer="19" extent="1-1"/>
+<wire x1="40.9575" y1="40.64" x2="41.275" y2="44.1325" width="0" layer="19" extent="1-1"/>
+<wire x1="39.0525" y1="40.005" x2="40.9575" y2="40.64" width="0" layer="19" extent="1-1"/>
+<wire x1="56.515" y1="34.075" x2="54.45125" y2="31.2175" width="0" layer="19" extent="1-1"/>
+<wire x1="37.25" y1="36.5125" x2="35.8775" y2="40.005" width="0" layer="19" extent="1-1"/>
+<wire x1="43.815" y1="26.1375" x2="44.74" y2="30.04" width="0" layer="19" extent="1-1"/>
+<wire x1="45.935" y1="20.32" x2="45.72" y2="25.0825" width="0" layer="19" extent="1-1"/>
+<wire x1="54.045" y1="18.77" x2="53.34" y2="20.6375" width="0" layer="19" extent="1-1"/>
+<wire x1="45.935" y1="17.78" x2="45.935" y2="20.32" width="0" layer="19" extent="1-1"/>
+<wire x1="59.905" y1="18.2" x2="56.445" y2="17.78" width="0" layer="19" extent="1-1"/>
+<wire x1="59.905" y1="21.2725" x2="59.905" y2="18.415" width="0" layer="19" extent="1-1"/>
+<wire x1="59.905" y1="14.2875" x2="60.325" y2="17.78" width="0" layer="19" extent="1-1"/>
+<wire x1="56.515" y1="24.765" x2="60.325" y2="21.9075" width="0" layer="19" extent="1-1"/>
+<wire x1="49.8475" y1="45.87875" x2="46.4575" y2="41.91" width="0" layer="19" extent="1-1"/>
+<wire x1="49.2506" y1="46.7106" x2="49.8475" y2="45.87875" width="0" layer="19" extent="1-1"/>
+<wire x1="51.91125" y1="56.99125" x2="51.22" y2="62.23" width="0" layer="19" extent="1-1"/>
+<wire x1="59.055" y1="56.515" x2="54.19" y2="56.3" width="0" layer="19" extent="1-1"/>
+<wire x1="56.73" y1="41.275" x2="52.705" y2="44.7675" width="0" layer="19" extent="1-1"/>
+<wire x1="59.905" y1="7.9375" x2="60.325" y2="13.6525" width="0" layer="19" extent="1-1"/>
+<wire x1="37.465" y1="29.63" x2="36.5125" y2="35.56" width="0" layer="19" extent="1-1"/>
+<wire x1="37.25" y1="23.495" x2="36.83" y2="28.575" width="0" layer="19" extent="1-1"/>
+<wire x1="57.15" y1="1.905" x2="60.325" y2="7.3025" width="0" layer="19" extent="1-1"/>
+<wire x1="49.8475" y1="1.27" x2="57.15" y2="1.905" width="0" layer="19" extent="1-1"/>
+<wire x1="45.085" y1="5.96" x2="49.8475" y2="2.72" width="0" layer="19" extent="1-1"/>
+<wire x1="46.0375" y1="7.62" x2="45.085" y2="6.6675" width="0" layer="19" extent="1-1"/>
+<wire x1="42.8625" y1="5.715" x2="45.085" y2="5.96" width="0" layer="19" extent="1-1"/>
+<wire x1="41.5925" y1="8.89" x2="41.91" y2="5.7875" width="0" layer="19" extent="1-1"/>
+<wire x1="38.1" y1="10.16" x2="39.6875" y2="8.89" width="0" layer="19" extent="1-1"/>
+<wire x1="38.1" y1="7.62" x2="39.6875" y2="8.89" width="0" layer="19" extent="1-1"/>
+<wire x1="35.56" y1="10.16" x2="38.1" y2="10.16" width="0" layer="19" extent="1-1"/>
+<wire x1="38.1" y1="5.08" x2="38.1" y2="7.62" width="0" layer="19" extent="1-1"/>
+<wire x1="35.56" y1="7.62" x2="38.1" y2="7.62" width="0" layer="19" extent="1-1"/>
+<wire x1="35.56" y1="5.08" x2="38.1" y2="5.08" width="0" layer="19" extent="1-1"/>
+<wire x1="-1.69" y1="-8.89" x2="35.56" y2="5.08" width="0" layer="19" extent="1-1"/>
+<wire x1="-1.69" y1="-12.065" x2="-1.69" y2="-8.89" width="0" layer="19" extent="1-1"/>
+<wire x1="-1.69" y1="-15.24" x2="-1.69" y2="-12.065" width="0" layer="19" extent="1-1"/>
 </signal>
 <signal name="-12V">
@@
 <wire x1="54.6625" y1="7.9375" x2="56.1725" y2="9.4475" width="0.4064" layer="1"/>
 </signal>
+<signal name="N$2">
+<contactref element="U1" pad="10"/>
+<contactref element="C34" pad="1"/>
+<wire x1="-3.39" y1="-15.24" x2="51.24" y2="36.04" width="0" layer="19" extent="1-1"/>
+</signal>
+<signal name="N$4">
+<contactref element="U1" pad="11"/>
+<contactref element="C33" pad="1"/>
+<wire x1="-3.39" y1="-12.065" x2="51.24" y2="36.54" width="0" layer="19" extent="1-1"/>
+</signal>
+<signal name="N$5">
+<contactref element="U1" pad="12"/>
+<contactref element="C32" pad="1"/>
+<wire x1="-3.39" y1="-8.89" x2="51.24" y2="37.04" width="0" layer="19" extent="1-1"/>
+</signal>
 </signals>
