File: BalancedIO/schematics/DualBalancedOutput.brd (EAGLE design)
At the start: 49.5 x 48.6 mm, 30 parts, among them IC1 THAT1646, IC2 THAT1646, J1 CON-JST_PH_3W

Commit message: set resistor values for voltage divider
Parts:
- R1, R3: value (none) -> 1k
- R2, R4: value (none) -> 220R
Changed lines of the file:
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@@
 <attribute name="VALUE" x="9.779" y="20.066" size="1.27" layer="27" ratio="10" rot="R90"/>
 </element>
-<element name="R1" library="Rebel" package="0204/7" value="" x="10.795" y="6.985" smashed="yes">
+<element name="R1" library="Rebel" package="0204/7" value="1k" x="10.795" y="6.985" smashed="yes">
 <attribute name="NAME" x="9.8425" y="6.477" size="1.016" layer="25" font="vector" ratio="10"/>
 <attribute name="VALUE" x="8.509" y="6.4262" size="1.27" layer="27" ratio="10"/>
 </element>
-<element name="R3" library="Rebel" package="0204/7" value="" x="10.795" y="4.445" smashed="yes">
+<element name="R3" library="Rebel" package="0204/7" value="1k" x="10.795" y="4.445" smashed="yes">
 <attribute name="NAME" x="9.8425" y="3.937" size="1.016" layer="25" font="vector" ratio="10"/>
 <attribute name="VALUE" x="8.509" y="3.8862" size="1.27" layer="27" ratio="10"/>
 </element>
-<element name="R4" library="Rebel" package="0204/7" value="" x="24.765" y="17.145" smashed="yes">
+<element name="R4" library="Rebel" package="0204/7" value="220R" x="24.765" y="17.145" smashed="yes">
 <attribute name="NAME" x="23.8125" y="16.637" size="1.016" layer="25" font="vector" ratio="10"/>
 <attribute name="VALUE" x="22.479" y="16.5862" size="1.27" layer="27" ratio="10"/>
 </element>
-<element name="R2" library="Rebel" package="0204/7" value="" x="24.765" y="19.05" smashed="yes">
+<element name="R2" library="Rebel" package="0204/7" value="220R" x="24.765" y="19.05" smashed="yes">
 <attribute name="NAME" x="23.8125" y="18.542" size="1.016" layer="25" font="vector" ratio="10"/>
 <attribute name="VALUE" x="22.479" y="18.4912" size="1.27" layer="27" ratio="10"/>
