File: QuantumEntaglement/schematics/QuantumEntanglement.sch (EAGLE design)
At the start: 4 parts, among them IC4 TL072D

Commit message: work in progress
Parts:
- added BOOT: (no value), SparkFun:M03PTH
- added C1, C500, C501: 100n, resistor:C-EUC0603
- added CV_C, CV_D, FREQ_X, FREQ_Y: THONKICONN, Rebel:THONKICONN
- added D600, D700, D800: BAT54S, diode:BAT54S
- added IC1: TL074D, linear:TL074D
- added IC2: QUAD_OPAMPD, adafruit:QUAD_OPAMPD
- added JP8: M05X2PTH, SparkFun:M05X2PTH
- added POT_A, POT_B, POT_C, POT_D: POT-ALPS-RK09L1140, Rebel:POT-ALPS-RK09L1140
- added Q1: SI2309CDS, transistor-small-signal:BSS84
- added Q2: BSS123, transistor-small-signal:BSS123
- added R1, R2, R3, R4, R5, R500, R501, R6, R600, R601, R7, R700, R701, R800, R801: 100k, Rebel:R-EU_0603
- added R15: 150R, Rebel:R-EU_0603
- added R503, R603, R703, R803: 33k, Rebel:R-EU_0603
- added R504, R604, R704, R804: 1k, Rebel:R-EU_0603
- added R605, R705, R805: 100R, Rebel:R-EU_0603
- IC4: value TL072D -> LM4040B10; device linear:TL072D -> texas:LM4041C12DBZ
Connections:
- new net +3V3: BOOT.3, D600.C2, D700.C2, D800.C2
- new net -12V: C501.2, IC2E.V-, IC2P.V-, Q1.C, Q2.S, R15.1, R3.2
- new net ADC3: R705.1
- new net ADC4: R805.1
- new net BOOT0: BOOT.2
- new net CV_REF: C1.1, IC4.A, POT_AG$1.1, POT_BG$1.1, POT_CG$1.1, POT_DG$1.1, R15.2
- new net FM_IN: R15.1
- new net FREQ_IN: IC1G$1.15, R5.1, R7.1
- new net FREQ_X: R504.1
- new net FREQ_Y: R605.1
- new net IC2_11: R3.1
- new net IC2_3: R15.1
- new net IC2_4: R3.2
- new net IC2_5: R15.2
- new net IN_A: R1.1
- new net IN_C: R7.1
- new net IN_D: R4.1
- new net N$1: IC1G$1.1, IC2A.CTRL, R1.1, R1.2, R7.2
- new net N$10: IC1G$1.8, R5.2, R6.2
- new net N$11: IC1G$1.9
- new net N$12: IC2B.IN, JP8.1, JP8.2, Q1.B, Q1.D
- new net N$13: IC2A.-IN, R500.2, R501.2, R503.1
- new net N$14: IC1G$1.11, IC2D.CTRL, POT_AG$1.2, R500.1
- new net N$16: IC1G$1.14
- new net N$17: IC1G$1.13, IC2A.OUT, IC2E.MODE, R15.2, R503.2, R504.2
- new net N$19: FREQ_Y.3, R601.1
- new net N$2: C1.1, IC1D.-IN, R1.1, R1.2, R2.2, R5.1, R6.1
- new net N$20: IC2B.-IN, R600.2, R601.2, R603.1
- new net N$21: POT_BG$1.2, R600.1
- new net N$22: IC2B.OUT, R603.2, R604.2
- new net N$23: D600.C1A2, IC2C.IN, R604.1, R605.2, R7.2
- new net N$25: CV_C.3, R701.1
- new net N$27: POT_CG$1.2, R700.1
- new net N$28: IC2C.OUT, R703.2, R704.2
- new net N$29: D700.C1A2, R704.1, R705.2
- new net N$3: FREQ_X.3, IC1G$1.7, R2.1, R501.1
- new net N$31: CV_D.3, R801.1
- new net N$33: IC2D.-IN, R800.2, R801.2, R803.1
- new net N$34: POT_DG$1.2, R800.1
- new net N$35: IC2D.OUT, R803.2, R804.2
- new net N$36: D800.C1A2, R804.1, R805.2
- new net N$4: IC1G$1.2, IC2D.IN, R2.1, R4.2, R5.2
- new net N$5: IC1C.-IN, IC1G$1.3, IC2A.IN, R1.2, R2.2, R3.1, R3.2, R4.1, R5.1
- new net N$6: IC2C.-IN, R5.2, R700.2, R701.2, R703.1
- new net N$7: IC2B.CTRL
- new net N$8: IC2C.CTRL, JP8.10, JP8.9, Q2.D
- new net N$9: C1.1, R7.2
- new net OUT_A: IC2A.OUT
- new net OUT_B: IC2B.OUT
- new net OUT_C: IC2C.OUT
- new net OUT_D: IC2D.OUT
- new net OUT_Y: IC1C.OUT, R3.1
- new net PULSE_OUT: IC1G$1.4, R4.1
- new net PWM_IN: IC1G$1.5
- new net TRI_OUT: IC1G$1.10, Q1.E
- new net VCA_IN_B: IC1D.OUT, R2.1
- new net VCA_IN_D: R7.1
- new net VCA_OUT_B: R4.2
- net +12V: now also C500.1, IC1G$1.16, IC2E.V+, IC2P.V+, Q1.S
- net CLAMP_REF: now also IC1A.-IN, IC1A.OUT; no longer IC4B.-IN, IC4B.OUT
- net GND: now also BOOT.1, C1.2, C500.2, C501.1, CV_C.4, CV_C.5, CV_D.4, CV_D.5, D600.A1, D700.A1, D800.A1, FREQ_X.4, FREQ_X.5, FREQ_Y.4, FREQ_Y.5, IC1C.+IN, IC1D.+IN, IC1G$1.12, IC2A.+IN, IC2B.+IN, IC2C.+IN, IC2D.+IN, IC2E.GND, IC4.C, JP8.3, JP8.4, JP8.5, JP8.6, JP8.7, JP8.8, POT_AG$1.3, POT_BG$1.3, POT_CG$1.3, POT_DG$1.3, Q1.G, Q2.G, R4.2
- net N$78: now also IC1A.+IN; no longer IC4B.+IN
Other:
- note added: "-10V"
- note added: "Crossfade Tri and Ramp. TODO: adjust for difference in output levels. TODO: convert VCA output from current to voltage"
- note added: "FM amount controlled by VCA CV. TODO: convert VCA output from current to voltage"
