File: TapTempo/schematics/TapTempoMk2.sch (EAGLE design)
At the start: 72 parts, among them IC1 TLV1117-33CDCY, IC2 TL072D, IC3 LM4040B10, P1 POT-ALPS-RK09L1140, P2 POT-ALPS-RK09L1140, SW1 SUB-MIN-SPDT, SW2 SUB-MIN-SPDT, T1 BC846, T2 BC846, T3 BC846, T4 BC846, U1 STM32F100CBT6B, X1 53048-05, Y1 8MHz

Commit message: rev06
Parts:
- removed D1, D2: (no value), SparkFun:DIODESMA
- added Q4: SI2309CDS, transistor-small-signal:BSS84
- added Q5: BSS123, transistor-small-signal:BSS123
- C12, C17: device resistor:CPOL-EUA -> Rebel:CPOL-EU153CLV-0405
- R22: value 20k -> 6k8
Connections:
- net +12V: now also Q4.S; no longer D1.C
- net -12V: now also Q5.S; no longer D2.A
- net GND: now also Q4.G, Q5.G
- net N$16: now also Q5.D; no longer D2.C
- net N$6: now also Q4.D; no longer D1.A
Other:
- note added: "Rebel Technology TapTempo Rev06"
- note removed: "Rebel Technology TapTempo Rev05"
Changed lines of the file:
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@@
 <part name="GND15" library="supply1" deviceset="GND" device=""/>
 <part name="GND10" library="supply1" deviceset="GND" device=""/>
-<part name="P+3" library="supply1" deviceset="+12V" device=""/>
-<part name="D1" library="SparkFun" deviceset="DIODE" device="SMA"/>
 <part name="GND28" library="supply1" deviceset="GND" device=""/>
-<part name="D2" library="SparkFun" deviceset="DIODE" device="SMA"/>
-<part name="P-1" library="supply1" deviceset="-12V" device=""/>
 <part name="R26" library="Rebel" deviceset="R-EU_" device="0603" value="100R"/>
 <part name="TEMPO1" library="Rebel" deviceset="THONKICONN" device=""/>
 <part name="DAC1" library="Rebel" deviceset="THONKICONN" device=""/>
-<part name="R22" library="Rebel" deviceset="R-EU_" device="0603" value="20k"/>
+<part name="R22" library="Rebel" deviceset="R-EU_" device="0603" value="6k8"/>
 <part name="R24" library="Rebel" deviceset="R-EU_" device="0603" value="3k3"/>
 <part name="GND44" library="supply1" deviceset="GND" device=""/>
@@
 <part name="GND43" library="supply1" deviceset="GND" device=""/>
 <part name="GND37" library="supply1" deviceset="GND" device=""/>
-<part name="C12" library="resistor" deviceset="CPOL-EU" device="A" value="10u">
+<part name="C12" library="Rebel" deviceset="CPOL-EU" device="153CLV-0405" value="10u">
 <attribute name="FARNELL" value="882-3014"/>
 </part>
-<part name="C17" library="resistor" deviceset="CPOL-EU" device="A" value="10u">
+<part name="C17" library="Rebel" deviceset="CPOL-EU" device="153CLV-0405" value="10u">
 <attribute name="FARNELL" value="882-3014"/>
 </part>
@@
 <part name="C19" library="Rebel" deviceset="C-EU" device="C0603" value="100n"/>
 <part name="GND48" library="supply1" deviceset="GND" device=""/>
+<part name="P+6" library="supply1" deviceset="+12V" device=""/>
+<part name="P-4" library="supply1" deviceset="-12V" device=""/>
+<part name="Q4" library="transistor-small-signal" deviceset="BSS84" device="" value="SI2309CDS">
+<attribute name="OC_FARNELL" value="1779264"/>
+</part>
+<part name="Q5" library="transistor-small-signal" deviceset="BSS123" device="">
+<attribute name="OC_FARNELL" value="1843725"/>
+</part>
 </parts>
 <sheets>
 <sheet>
 <plain>
-<text x="-114.3" y="-12.7" size="3.048" layer="97" font="vector">Rebel Technology TapTempo Rev05</text>
+<text x="-114.3" y="-12.7" size="3.048" layer="97" font="vector">Rebel Technology TapTempo Rev06</text>
 <text x="-114.3" y="-22.86" size="3.048" layer="97" font="vector">Published 2017 under the GNU GPL v2</text>
 <text x="170.18" y="10.16" size="1.778" layer="97">LP Fc apprx 800Hz</text>
@@
 <instance part="GND15" gate="1" x="2.54" y="81.28"/>
 <instance part="GND10" gate="1" x="-17.78" y="81.28"/>
-<instance part="P+3" gate="1" x="127" y="114.3"/>
-<instance part="D1" gate="G$1" x="119.38" y="104.14"/>
 <instance part="GND28" gate="1" x="93.98" y="83.82"/>
-<instance part="D2" gate="G$1" x="119.38" y="93.98" rot="R180"/>
-<instance part="P-1" gate="1" x="127" y="83.82"/>
 <instance part="R26" gate="G$1" x="172.72" y="48.26"/>
 <instance part="TEMPO1" gate="G$1" x="-27.94" y="99.06" rot="R180"/>
@@
 <instance part="C19" gate="G$1" x="190.5" y="116.84" rot="R90"/>
 <instance part="GND48" gate="1" x="198.12" y="91.44"/>
+<instance part="P+6" gate="1" x="124.46" y="114.3"/>
+<instance part="P-4" gate="1" x="124.46" y="83.82"/>
+<instance part="Q4" gate="G$1" x="116.84" y="104.14" rot="MR90">
+<attribute name="OC_FARNELL" x="116.84" y="104.14" size="1.778" layer="96" rot="MR90" display="off"/>
+</instance>
+<instance part="Q5" gate="G$1" x="116.84" y="93.98" rot="MR270">
+<attribute name="OC_FARNELL" x="116.84" y="93.98" size="1.778" layer="96" rot="MR270" display="off"/>
+</instance>
 </instances>
 <busses>
@@
 <nets>
 <net name="+12V" class="0">
-<segment>
-<pinref part="P+3" gate="1" pin="+12V"/>
-<wire x1="127" y1="111.76" x2="127" y2="104.14" width="0.1524" layer="91"/>
-<wire x1="121.92" y1="104.14" x2="127" y2="104.14" width="0.1524" layer="91"/>
-<pinref part="D1" gate="G$1" pin="C"/>
-</segment>
 <segment>
 <pinref part="R10" gate="G$1" pin="1"/>
@@
 <junction x="134.62" y="180.34"/>
 <pinref part="P+4" gate="1" pin="+12V"/>
+</segment>
+<segment>
+<pinref part="P+6" gate="1" pin="+12V"/>
+<wire x1="124.46" y1="111.76" x2="124.46" y2="104.14" width="0.1524" layer="91"/>
+<wire x1="124.46" y1="104.14" x2="121.92" y2="104.14" width="0.1524" layer="91"/>
+<pinref part="Q4" gate="G$1" pin="S"/>
 </segment>
 </net>
@@
 <wire x1="111.76" y1="101.6" x2="96.52" y2="101.6" width="0.1524" layer="91"/>
 <junction x="96.52" y="101.6"/>
+<pinref part="Q4" gate="G$1" pin="G"/>
+<pinref part="Q5" gate="G$1" pin="G"/>
+<wire x1="111.76" y1="99.06" x2="119.38" y2="99.06" width="0.1524" layer="91"/>
+<junction x="111.76" y="99.06"/>
+<junction x="119.38" y="99.06"/>
 </segment>
 <segment>
@@
 <net name="-12V" class="0">
 <segment>
-<wire x1="127" y1="93.98" x2="127" y2="86.36" width="0.1524" layer="91"/>
-<pinref part="P-1" gate="1" pin="-12V"/>
-<pinref part="D2" gate="G$1" pin="A"/>
-<wire x1="121.92" y1="93.98" x2="127" y2="93.98" width="0.1524" layer="91"/>
-</segment>
-<segment>
 <pinref part="IC2" gate="P" pin="V-"/>
 <pinref part="P-3" gate="1" pin="-12V"/>
@@
 <pinref part="R21" gate="G$1" pin="1"/>
 <wire x1="142.24" y1="132.08" x2="142.24" y2="129.54" width="0.1524" layer="91"/>
+</segment>
+<segment>
+<wire x1="121.92" y1="93.98" x2="124.46" y2="93.98" width="0.1524" layer="91"/>
+<wire x1="124.46" y1="93.98" x2="124.46" y2="86.36" width="0.1524" layer="91"/>
+<pinref part="P-4" gate="1" pin="-12V"/>
+<pinref part="Q5" gate="G$1" pin="S"/>
 </segment>
 </net>
@@
 <pinref part="SV1" gate="G$1" pin="9"/>
 <wire x1="96.52" y1="104.14" x2="111.76" y2="104.14" width="0.1524" layer="91"/>
-<pinref part="D1" gate="G$1" pin="A"/>
-<wire x1="111.76" y1="104.14" x2="116.84" y2="104.14" width="0.1524" layer="91"/>
 <junction x="111.76" y="104.14"/>
+<pinref part="Q4" gate="G$1" pin="D"/>
 </segment>
 </net>
@@
 <pinref part="SV1" gate="G$1" pin="1"/>
 <wire x1="96.52" y1="93.98" x2="111.76" y2="93.98" width="0.1524" layer="91"/>
-<pinref part="D2" gate="G$1" pin="C"/>
-<wire x1="111.76" y1="93.98" x2="116.84" y2="93.98" width="0.1524" layer="91"/>
 <junction x="111.76" y="93.98"/>
-</segment>
-</net>
+<pinref part="Q5" gate="G$1" pin="D"/>
+</segment>
+</net>

Commit message: updated for publishing schematics
Other:
- note added: "Rebel Technology TapTempo mkII Rev06"
- note removed: "Rebel Technology TapTempo Rev06"
