File: Wizard/schematics/Witch.brd (EAGLE design)
At the start: 231 x 94 mm, 115 parts, among them IC1 TS924, J1 THONKICONN, J2 THONKICONN, J3 THONKICONN, J4 THONKICONN, J5 THONKICONN, J6 THONKICONN, J7 POWER_JACK, P1 POT-ALPS-RK09L1140, P2 POT-ALPS-RK09L1140, P3 POT-ALPS-RK09L1140, P4 POT-ALPS-RK09L1140, P5 POT-ALPS-RK09L1140, T1 2N3904, U2 LM7805, X3 KUSBVX, X5 USBPTH-VERTICAL

Commit message: Witch is not Wizard
Parts:
- removed JP13: (no value), jumper:JP1
- removed LED1: MULTICOMP_703-1028, Rebel:RGB-LED-703-1028
- removed R11: 510R, Rebel:0204/7
- added C24, C26, C27, C28: 100n, resistor:C050-024X044
- added D2, D3, D8, D9: 1N5818-T, diode:DO41-7.6
- added IC2: OPAMP-DUALDIP, SparkFun:DIP08
- added J10, J11, J12, J13, J8, J9: THONKICONN, Rebel:THONKICONN
- added LED2, LED3, LED4, LED5, LED6, LED7, LED8, LED9: (no value), Rebel:LED3MM
- added R19, R44, R47: 100k, Rebel:0204/7
- added R20, R45, R48: 1M, Rebel:0204/7
- added R4, R43, R46, R49, R50, R54, R60, R63, R75, R76, R77: 1k, Rebel:0204/7
- added R55, R56, R61, R62, R64, R65: 10k, Rebel:0204/7
- added R57, R67, R68, R71, R74: 100R, Rebel:0204/7
- added R58, R59, R70, R73: 51k, Rebel:0204/7
- added R66: 5k1, Rebel:0204/7
- added R69, R72: 33k, Rebel:0204/7
- added T2, T3, T4, T5, T6, T7, T8: 2N3904, transistor-npn:TO92
- R12, R17: value 1k -> 100R
- R18: value 1k -> 5k1
- R39: value 220R -> 100R
- R40: value 220R -> 1k
- R41, R42: value 5k1 -> 33k
- SW1, SW2, SW3, SW4: value (none) -> PB6146L; device switch-omron:B3F-10XX -> Rebel:PB6146L
- moved D7 192.5 mm to (-39.4, -64.8), turned to 0 degrees
- moved D5 189.7 mm to (-80.0, -38.1), turned to 180 degrees
- moved D6 181.9 mm to (-39.4, -57.1), turned to 0 degrees
- moved D4 181.5 mm to (-80.0, -34.3), turned to 180 degrees
- moved R40 180.7 mm to (-120.7, -27.9), flipped to the top
- moved R39 162.5 mm to (-105.4, -20.3), flipped to the top
- moved R17 148.7 mm to (-45.1, 63.5), flipped to the top, turned to 90 degrees
- moved R12 137.6 mm to (-38.7, -10.2), flipped to the top
- moved J5 134.0 mm to (-38.7, 6.35)
- moved J6 129.8 mm to (-24.8, 64.8)
- moved SW5 128.8 mm to (-31.8, 44.5)
- moved R7 118.0 mm to (10.2, -59.7), flipped to the top
- moved J4 116.0 mm to (-38.7, 64.8)
- moved C13 112.2 mm to (16.5, -35.6), flipped to the top
- moved C16 110.3 mm to (19.1, -43.2), flipped to the top
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Connections:
- removed net A18_ADC1: JP7.4, P3.2
- removed net A19_ADC2: D4.A, D5.C, JP7.3, P2.2
- removed net A20_ADC3: D6.A, D7.C, JP7.2, P1.2
- removed net A21_ADC4: JP7.1, P5.2
- removed net A23_ADC5: JP6.3, P4.2
- removed net N$18: JP13.2, X5.VBUS
- new net A13_TR_OUT1: R61.2
- new net A18_ADC: C26.1, JP7.4, R68.2
- new net A19_ADC: JP7.3, P1.2
- new net A1_ADC: C27.1, JP3.1, R71.2
- new net A20_ADC: C24.1, JP7.2, R57.2
- new net A21_ADC: JP7.1, P2.2
- new net A23_ADC: JP6.3, P5.2
- new net A2_ADC: JP3.2, P3.2
- new net A3_ADC: C28.1, JP3.3, R74.2
- new net A4_ADC: JP3.4, P4.2
- new net N$28: R4.2, SW1.PL1
- new net N$29: R19.2, R20.2, T2.2
- new net N$34: J8.P$3, R19.1
- new net N$35: R43.2, SW2.PL1
- new net N$36: R44.2, R45.2, T3.2
- new net N$38: J9.P$3, R44.1
- new net N$40: R46.2, SW3.PL1
- new net N$42: R47.2, R48.2, T4.2
- new net N$43: J10.P$3, R47.1
- new net N$44: R49.2, SW4.PL1
- new net N$45: LED2.A, R50.2
- new net N$49: LED6.A, T7.3
- new net N$50: R56.1, T7.2
- new net N$51: R60.2, T7.1
- new net N$52: D2.A, D3.C, R42.2, R58.1, R68.1
- new net N$53: J13.P$3, R69.1
- new net N$54: R61.1, T6.2
- new net N$55: LED7.A, T8.3
- new net N$56: R62.1, T8.2
- new net N$57: R63.2, T8.1
- new net N$58: D6.A, D7.C, R69.2, R70.1, R71.1
- new net N$59: J12.P$3, R72.1
- new net N$60: J4.P$3, R17.2
- new net N$61: IC2.6, R65.2, R66.2
- new net N$62: IC2.7, R66.1, R67.1
- new net N$63: J6.P$3, R67.2
- new net N$64: D8.A, D9.C, R72.2, R73.1, R74.1
- new net N$65: LED3.A, R75.2
- new net N$66: LED4.A, R76.2
- new net N$67: LED5.A, R77.2
- net +3V3: now also D2.C, D8.C, P1.3, P2.3
- net +5V: now also IC2.8, LED8.A, LED9.A, R4.1, R43.1, R46.1, R49.1, R50.1, R54.1, R60.1, R63.1, R75.1, R76.1, R77.1; no longer LED1.P3, R39.1
- net A13_TR_OUT: now also R55.2; no longer R12.2
- net A14_SW2: no longer SW2.1, SW2.2
- net A16_LEDPWM3: no longer R11.1
- net A17_SW1: now also SW1.P3, SW1.P4, SW1.PL2, SW2.P3, SW2.P4, SW2.PL2, SW3.P3, SW3.P4, SW3.PL2, SW4.P3, SW4.P4, SW4.PL2, T2.1, T3.1, T4.1; no longer SW1.1, SW1.2
- net A1_LEDPWM1: no longer JP3.1
- net A22_DAC2: now also IC2.5; no longer R17.2
- net A2_LEDPWM2: now also LED2.K, LED3.K, LED4.K, LED5.K; no longer JP3.2
- net A3_USART_TX: no longer JP3.3
- net A4_USART_RX: no longer JP3.4
- net A5_DAC1: now also IC2.3; no longer R18.2
- net A6_SW3: no longer SW3.1, SW3.2
- net A7_SW4: no longer SW4.1, SW4.2
- net GND: now also C24.2, C26.2, C27.2, C28.2, D3.A, D9.A, IC2.4, J1.P$2, J10.P$1, J11.P$1, J11.P$2, J12.P$1, J12.P$2, J13.P$1, J13.P$2, J3.P$2, J8.P$1, J9.P$1, LED6.K, LED7.K, R20.1, R45.1, R48.1, R58.2, R59.2, R64.1, R65.1, R70.2, R73.2, SW1.P1, SW1.P2, SW2.P1, SW2.P2, SW3.P1, SW3.P2, SW4.P1, SW4.P2, T2.3, T3.3, T4.3, T5.3, T6.3; no longer SW1.3, SW1.4, SW2.3, SW2.4, SW3.3, SW3.4, SW4.3, SW4.4
- net N$14: now also LED8.K, R10.2; no longer LED1.P2, R11.2
- net N$16: now also LED9.K; no longer LED1.P1
- net N$17: now also D4.A, D5.C, R41.2, R57.1, R59.1; no longer LED1.P4, R10.2
- net N$2: now also J11.P$3, R39.1; no longer J1.P$2, R40.2
- net N$20: now also IC2.2, R18.1, R64.2; no longer J6.P$3, R17.1
- net N$21: now also IC2.1, R17.1, R18.2; no longer J4.P$3, R18.1
- net N$23: now also R54.2, R62.2, T6.1; no longer J3.P$2
- net N$25: now also R12.2, R40.2, R56.2, T5.1; no longer P2.3, R41.2
- net N$31: now also R55.1, T5.2; no longer P1.3, R42.2
- net USBD_VBUS: now also X5.VBUS; no longer JP13.1
Other:
- board size 231 x 94 mm -> 295.8 x 94 mm
- board text removed: "3v3"
- board text removed: "5v"
- board text removed: "gnd"

Commit message: witch updates
Parts:
- removed C13: 22u, Rebel:E5-6
- removed C16: 100n, Rebel:C050-024X044
- removed C7: 10u, Rebel:E5-6
- removed C8: 100n 16v, Rebel:C050-024X044
- removed D1: (no value), Rebel:DIODE-1N4001
- removed J7: POWER_JACK, Rebel:DC_JACK_SLOT
- removed R56, R62: 10k, Rebel:0204/7
- removed T7, T8: 2N3904, transistor-npn:TO92
- removed U2: LM7805, Rebel:REG_S9V11F5
- moved VBUS 9.67 mm to (-53.6, 78.2)
- moved SW5 2.54 mm to (-31.8, 41.9)
- moved J11 2.54 mm to (-24.8, 8.89), turned to 90 degrees
- moved J5 2.54 mm to (-38.7, 8.89), turned to 270 degrees
- moved LED2 2.54 mm to (-69.8, 47.0)
- moved LED3 2.54 mm to (-55.9, 47.0)
- moved LED4 2.54 mm to (-7.62, 47.0)
- moved LED5 2.54 mm to (6.35, 47.0)
- moved LED8 2.54 mm to (-38.7, 57.1)
- moved LED9 2.54 mm to (-24.8, 57.1)
- turned J1 to 270 degrees
- turned J12 to 90 degrees
- turned J13 to 270 degrees
- turned J3 to 90 degrees
- turned J4 to 270 degrees
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Connections:
- removed net +9V: D1.A, J7.PWR
- removed net N$49: LED6.A, T7.3
- removed net N$50: R56.1, T7.2
- removed net N$51: R60.2, T7.1
- removed net N$55: LED7.A, T8.3
- removed net N$56: R62.1, T8.2
- removed net N$57: R63.2, T8.1
- new net N$18: LED7.K, R63.1
- new net N$46: LED6.K, R60.1
- net +5V: now also LED6.A, LED7.A; no longer C13.+, C16.1, R60.1, R63.1, U2.VOUT
- net +VIN: no longer C7.+, C8.1, D1.C, U2.VIN
- net A13_TR_OUT: now also R60.2
- net A13_TR_OUT1: now also R63.2
- net GND: no longer C13.-, C16.2, C7.-, C8.2, J7.GND, LED6.K, LED7.K, U2.GND
- net N$23: no longer R62.2
- net N$25: no longer R56.2
