File: Xibeca/schematics/Xibeca00.brd (EAGLE design)
At the start: 27.9 x 43.8 mm, 40 parts, among them IC1 STM32H743IIK6, IC2 AS4C16M32MSA-6BIN, IC9 S25FL064LABMFI010, J1 FTS-105-01-F-DV, U3 TLV1117LV33DCYR, Y1 8MHz

Commit message: wip
Changed lines of the file:
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@@
 <drawing>
 <settings>
-<setting alwaysvectorfont="yes"/>
+<setting alwaysvectorfont="no"/>
 <setting keepoldvectorfont="yes"/>
 <setting verticaltext="up"/>
@@
 <attribute name="NAME" x="7.6" y="37.0505" size="0.9" layer="25" font="vector" rot="R180" align="bottom-center"/>
 </element>
-<element name="R1" library="Rebel" library_urn="urn:adsk.eagle:library:15457297" package="R0402" package3d_urn="urn:adsk.eagle:package:26058/3" value="10k" x="23.65" y="36.35" smashed="yes" rot="R180"/>
+<element name="R1" library="Rebel" library_urn="urn:adsk.eagle:library:15457297" package="R0402" package3d_urn="urn:adsk.eagle:package:26058/3" value="10k" x="23.65" y="36.35" smashed="yes" rot="R180">
+<attribute name="NAME" x="22.959" y="36.929" size="0.8636" layer="25" font="vector"/>
+<attribute name="VALUE" x="24.285" y="38.255" size="1.27" layer="27" rot="R180"/>
+</element>
 <element name="BOOT" library="SparkFun" package="SJ_2S-NO" value="SOLDERJUMPERNO" x="22.575" y="36.8185" smashed="yes" rot="MR270">
 <attribute name="VALUE" x="24.226" y="37.9805" size="0.4064" layer="28" rot="MR270"/>
@@
 </element>
 <element name="L1" library="Rebel" library_urn="urn:adsk.eagle:library:15457297" package="0603" package3d_urn="urn:adsk.eagle:package:15457735/3" value="Ferrite Bead" x="6.25" y="22.6556" smashed="yes" rot="R90">
-<attribute name="NAME" x="6.399996875" y="24.217596875" size="0.9" layer="25" font="vector" align="bottom-center"/>
+<attribute name="NAME" x="8.076396875" y="22.134796875" size="0.9" layer="25" font="vector" align="bottom-center"/>
 <attribute name="OC_FARNELL" value="2288736" x="6.25" y="22.6556" size="1.778" layer="27" rot="R90" display="off"/>
 </element>
@@
 </element>
 <element name="C6" library="Rebel" library_urn="urn:adsk.eagle:library:15457297" package="C0402" package3d_urn="urn:adsk.eagle:package:15457953/1" value="100n" x="18.4" y="23.15" smashed="yes">
-<attribute name="NAME" x="19.715" y="22.685" size="0.9" layer="25" font="vector"/>
+<attribute name="NAME" x="19.8674" y="22.685" size="0.9" layer="25" font="vector"/>
 <attribute name="VALUE" x="17.765" y="21.245" size="1.27" layer="27"/>
 </element>
