File: Xibeca/schematics/Xibeca44.brd (EAGLE design)
At the start: 30 x 62 mm, 57 parts, among them IC1 STM32H743IIK6, IC2 AS4C16M32MSA-6BIN, IC3 CS4244, IC9 S25FL064LABMFI010, J1 FTS-105-01-F-DV, U3 TLV1117LV33DCYR, Y1 8MHz

Commit message: wip
Parts:
- moved R2 0.63 mm to (15.7, 21.5)
- moved R3 0.63 mm to (14.4, 21.5)
Routing:
- net ADC_I2C_SDA: track 26.5 -> 25.8 mm
- net ADC_I2C_SCL: track 29.1 -> 28.5 mm
